File: electronics/simplified/v1/simplified_spincoater_v1/Capacitor Bank.kicad_sch (KiCad schematic)
At the start: 20 parts

Commit message: fix
Parts:
- removed C34, C35, C36, C37, C38, C39, C40, C41, C42, C43, C44, C45, C46, C47, C48, C49, C50, C51, C52, C53: 4u7, Capacitor_SMD:C_0402_1005Metric, symbol Device:C
- added C14, C15, C16, C17, C18, C19, C20, C23, C28, C31, C32, C33: 10u, Capacitor_SMD:C_1210_3225Metric, symbol Device:C
Connections:
- net GND: now also C14.2, C15.2, C16.2, C17.2, C18.2, C19.2, C20.2, C23.2, C28.2, C31.2, C32.2, C33.2
- net VBUS: now also C14.1, C15.1, C16.1, C17.1, C18.1, C19.1, C20.1, C23.1, C28.1, C31.1, C32.1, C33.1
Other:
- note added: "10x 10u"
- note removed: "20x 4u7"
