File: electronics/simplified/v1/simplified_spincoater_v1/H-Bridge.kicad_sch (KiCad schematic)
At the start: 9 parts, among them U11 NTTFS5C454NL, U13 NTTFS5C454NL, U14 NTTFS5C454NL, U15 NTTFS5C454NL, U16 NTTFS5C454NL, U17 NTTFS5C454NL

Commit message: fix
Parts:
- removed R26, R27: 22r, Resistor_SMD:R_0201_0603Metric, symbol Device:R
- added R29, R30: 2m, Resistor_SMD:R_0612_1632Metric, symbol Device:R
- R28: value 22r -> 2m; footprint Resistor_SMD:R_0201_0603Metric -> Resistor_SMD:R_0612_1632Metric; Manufacturer (none) -> prosemi; Manufacturer Part Number (none) -> MLR06A1R002F2
- U11, U13, U14, U15, U16, U17: Manufacturer (none) -> onsemi; Manufacturer Part Number (none) -> NTTFS5C454NL
Connections:
- net GND: now also R29.1, R30.1
- net H_BRIDGE_SPA: now also R28.2
- net H_BRIDGE_SPB: now also R29.2
- net H_BRIDGE_SPC: now also R30.2; no longer R28.2
Other:
- moved on the sheet: R28

Commit message: fix
Parts:
- added J1: Screw_Terminal_01x03, symbol Connector:Screw_Terminal_01x03
Connections:
- net H_BRIDGE_SHA: now also J1.1 (Pin_1)
- net H_BRIDGE_SHB: now also J1.2 (Pin_2)
- net H_BRIDGE_SHC: now also J1.3 (Pin_3)
Changed lines of the file:
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@@
 	(wire
 		(pts
-			(xy 149.86 124.46) (xy 137.16 124.46)
+			(xy 149.86 127) (xy 137.16 127)
 		)
 		(stroke
@@
 	(wire
 		(pts
-			(xy 149.86 134.62) (xy 137.16 134.62)
+			(xy 149.86 132.08) (xy 137.16 132.08)
 		)
 		(stroke
@@
 	)
 	(label "MOTOR_C"
-		(at 137.16 134.62 0)
+		(at 137.16 132.08 0)
 		(effects
 			(font
@@
 	)
 	(label "MOTOR_A"
-		(at 137.16 124.46 0)
+		(at 137.16 127 0)
 		(effects
 			(font
@@
 					(unit 1)
 				)
+			)
+		)
+	)
+	(symbol
+		(lib_id "Connector:Screw_Terminal_01x03")
+		(at 154.94 129.54 0)
+		(unit 1)
+		(exclude_from_sim no)
+		(in_bom yes)
+		(on_board yes)
+		(dnp no)
+		(fields_autoplaced yes)
+		(property "Reference" "J1"
+			(at 157.48 128.2699 0)
+			(effects
+				(font
+					(size 1.27 1.27)
+				)
+				(justify left)
+			)
+		)
+		(property "Value" "Screw_Terminal_01x03"
+			(at 157.48 130.8099 0)
+			(effects
+				(font
+					(size 1.27 1.27)
+				)
+				(justify left)
+			)
+		)
+		(property "Footprint" ""
+			(at 154.94 129.54 0)
+			(effects
+				(font
+					(size 1.27 1.27)
+				)
+				(hide yes)
+			)
+		)
+		(property "Datasheet" "~"
+			(at 154.94 129.54 0)
+			(effects
+				(font
+					(size 1.27 1.27)
+				)
+				(hide yes)
+			)
+		)
+		(property "Description" "Generic screw terminal, single row, 01x03, script generated (kicad-library-utils/schlib/autogen/connector/)"
+			(at 154.94 129.54 0)
+			(effects
+				(font
+					(size 1.27 1.27)
+				)
+				(hide yes)
+			)
+		)
+		(pin "3"
+		)
+		(pin "2"
+		)
+		(pin "1"
+		)
+		(instances
+			(project ""
+				(path "/82f7d8d0-a6dd-48aa-80fa-49fc2cccb16f/c9ec9ccd-2e72-4236-908b-58c2b4d5f776/effaf589-d03b-428f-9cd2-be6913714a7d"
+					(reference "J1")
+					(unit 1)
+				)
