File: electronics/simplified/v1/simplified_spincoater_v1/MCU.kicad_sch (KiCad schematic)
At the start: 5 parts, among them U6 ESP32-S3-WROOM-1

Commit message: fix
Parts:
- removed C10, C12: 100n, Capacitor_SMD:C_0402_1005Metric, symbol Device:C
- removed C13: 1u, Capacitor_SMD:C_0402_1005Metric, symbol Device:C
- removed R14: 10k, Resistor_SMD:R_0201_0603Metric, symbol Device:R
- added C29: 1u, Capacitor_SMD:C_0402_1005Metric, symbol Device:C
- added C44, C56: 100n, Capacitor_SMD:C_0402_1005Metric, symbol Device:C
- added R38: 10k, Resistor_SMD:R_0402_1005Metric, symbol Device:R
- U6: Manufacturer (none) -> Espressif Systems; Manufacturer Part Number (none) -> ESP32-S3-WROOM-1
Connections:
- net +3V3: now also C29.1, C56.1, R38.1
- net GND: now also C29.2, C44.2, C56.2
- net at U6.3 (EN): now also C44.1, R38.2

Commit message: fix
Parts:
- added R39: 10k, Resistor_SMD:R_0402_1005Metric, symbol Device:R
- added S1, S2: TS-1088-AR02016, simplified_spincoater_v1:TS-1088-AR02016, symbol simplified_spincoater_v1:TS-1088-AR02016
Connections:
- net +3V3: now also R39.1
- net CAN_TX: now also U6.35 (IO42); no longer U6.16 (IO46)
- net EN_12V: now also U6.8 (IO15); no longer U6.33 (IO40)
- net GND: now also S1.2, S2.2
- net PD_FAULT: now also U6.16 (IO46); no longer U6.28 (IO35)
- net PD_INT_N: now also U6.15 (IO3); no longer U6.23 (IO21)
- net at U6.27 (IO0): now also R39.2, S2.1
- net at C44.1, R38.2, U6.3 (EN): now also S1.1
Other:
- moved on the sheet: C44, R38

Commit message: fix
Connections:
- net GND renamed EPAD
- net EPAD: now also U6.41_1 (EPAD), U6.41_2 (EPAD), U6.41_3 (EPAD), U6.41_4 (EPAD), U6.41_5 (EPAD), U6.41_6 (EPAD), U6.41_7 (EPAD), U6.41_8 (EPAD), U6.41_9 (EPAD)
Changed lines of the file:
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@@
 	(paper "A4")
+	(junction
+		(at 119.38 60.96)
+		(diameter 0)
+		(color 0 0 0 0)
+	)
 	(junction
 		(at 160.02 124.46)
@@
 	)
 	(junction
-		(at 119.38 60.96)
-		(diameter 0)
-		(color 0 0 0 0)
-	)
-	(junction
 		(at 109.22 60.96)
 		(diameter 0)
@@
 	(wire
 		(pts
+			(xy 157.48 124.46) (xy 160.02 124.46)
+		)
+		(stroke
+			(width 0)
+			(type default)
+		)
+	)
+	(wire
+		(pts
 			(xy 81.28 86.36) (xy 81.28 81.28)
 		)
@@
 	(wire
 		(pts
+			(xy 157.48 73.66) (xy 160.02 73.66)
+		)
+		(stroke
+			(width 0)
+			(type default)
+		)
+	)
+	(wire
+		(pts
+			(xy 99.06 91.44) (xy 99.06 93.98)
+		)
+		(stroke
+			(width 0)
+			(type default)
+		)
+	)
+	(wire
+		(pts
 			(xy 160.02 124.46) (xy 160.02 127)
 		)
@@
 	(wire
 		(pts
-			(xy 157.48 73.66) (xy 160.02 73.66)
-		)
-		(stroke
-			(width 0)
-			(type default)
-		)
-	)
-	(wire
-		(pts
-			(xy 99.06 91.44) (xy 99.06 93.98)
-		)
-		(stroke
-			(width 0)
-			(type default)
-		)
-	)
-	(wire
-		(pts
 			(xy 157.48 78.74) (xy 160.02 78.74)
 		)
@@
 		(pts
 			(xy 127 91.44) (xy 124.46 91.44)
-		)
-		(stroke
-			(width 0)
-			(type default)
-		)
-	)
-	(wire
-		(pts
-			(xy 157.48 124.46) (xy 160.02 124.46)
 		)
 		(stroke
@@
 		(pin "41"
 		)
+		(pin "41_1"
+		)
+		(pin "41_2"
+		)
+		(pin "41_3"
+		)
+		(pin "41_4"
+		)
+		(pin "41_5"
+		)
+		(pin "41_6"
+		)
+		(pin "41_7"
+		)
+		(pin "41_8"
+		)
+		(pin "41_9"
+		)
 		(instances
