File: electronics/simplified/v1/simplified_spincoater_v1/STM32.kicad_sch (KiCad schematic)
At the start: 9 parts, among them U7 STM32G474VEH6

Commit message: fix
Parts:
- removed C14, C15, C16, C17, C19, C20: 100n, Capacitor_SMD:C_0402_1005Metric, symbol Device:C
- removed C18: 1u, Capacitor_SMD:C_0402_1005Metric, symbol Device:C
- removed R15: 10k, Resistor_SMD:R_0201_0603Metric, symbol Device:R
- added C30: 1u, Capacitor_SMD:C_0402_1005Metric, symbol Device:C
- added C46, C47, C48, C49, C50, C51: 100n, Capacitor_SMD:C_0402_1005Metric, symbol Device:C
- added R21: 10k, Resistor_SMD:R_0402_1005Metric, symbol Device:R
- U7: Manufacturer (none) -> STMicroelectronics; Manufacturer Part Number (none) -> STM32G474VEH6
Connections:
- net +3V3: now also C30.1, C46.1, C47.1, C48.1, C49.1, C50.1, C51.1
- net GND: now also C30.2, C46.2, C47.2, C48.2, C49.2, C50.2, C51.2, R21.2
- net STM32_EN: now also R21.1

Commit message: fix
Connections:
- net GATE_DRIVER_NFALUT renamed GATE_DRIVER_NFAULT
Changed lines of the file:
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@@
 		)
 	)
-	(hierarchical_label "GATE_DRIVER_NFALUT"
+	(hierarchical_label "GATE_DRIVER_NFAULT"
 		(shape output)
 		(at 116.84 109.22 180)
