File: electronics/simplified/v1/simplified_spincoater_v1/motor.kicad_sch (KiCad schematic)
At the start: 0 parts

Commit message: fix
Other:
- sheet Gate Driver ports: added GATE_DRIVER_NFAULT; removed GATE_DRIVER_NFALUT
- sheet STM32 ports: added GATE_DRIVER_NFAULT; removed GATE_DRIVER_NFALUT
Changed lines of the file:
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@@
-			)
-		)
-		(pin "GATE_DRIVER_NFALUT" output
-			(at 134.62 86.36 180)
-			(effects
-				(font
-					(size 1.27 1.27)
-				)
-				(justify left)
 			)
 		)
@@
 		(pin "MOTOR_C_CURRENT_SENSE" output
 			(at 134.62 96.52 180)
+			(effects
+				(font
+					(size 1.27 1.27)
+				)
+				(justify left)
+			)
+		)
+		(pin "GATE_DRIVER_NFAULT" output
+			(at 134.62 86.36 180)
 			(effects
 				(font
@@
 			)
 		)
-		(pin "GATE_DRIVER_NFALUT" output
-			(at 119.38 86.36 0)
-			(effects
-				(font
-					(size 1.27 1.27)
-				)
-				(justify right)
-			)
-		)
 		(pin "GATE_DRIVER_NSCS" output
 			(at 119.38 81.28 0)
@@
 			)
 		)
+		(pin "GATE_DRIVER_NFAULT" output
+			(at 119.38 86.36 0)
+			(effects
+				(font
+					(size 1.27 1.27)
+				)
+				(justify right)
+			)
+		)
