File: electronics/simplified/v1/simplified_spincoater_v1/simplified_spincoater_v1.kicad_pcb (KiCad board)
At the start: 2 copper layers, 105 parts, among them U1 HUSB238A-BB001-QN16R, U10 TJA1051TK/3, U11 NTTFS5C454NL, U13 NTTFS5C454NL, U14 NTTFS5C454NL, U15 NTTFS5C454NL, U16 NTTFS5C454NL, U17 NTTFS5C454NL, U18 TJA1051TK/3, U2 LMR51420YDD, U3 TPS62933DRL, U4 GT-USB-7004N, U6 ESP32-S3-WROOM-1, U7 STM32G474VEH6, U8 DRV8323SRTA, U9 AS5600

Commit message: fix
Parts:
- added C14: 10u, Capacitor_SMD:C_1210_3225Metric, F.Cu at (2.33, 1.62)
- added C15: 10u, Capacitor_SMD:C_1210_3225Metric, F.Cu at (2.33, 5.88)
- added C16: 10u, Capacitor_SMD:C_1210_3225Metric, F.Cu at (2.33, 10.1)
- added C17: 10u, Capacitor_SMD:C_1210_3225Metric, F.Cu at (7.97, 1.62)
- added C18: 10u, Capacitor_SMD:C_1210_3225Metric, F.Cu at (7.97, 5.88)
- added C19: 10u, Capacitor_SMD:C_1210_3225Metric, F.Cu at (7.97, 10.1)
- added C20: 10u, Capacitor_SMD:C_1210_3225Metric, F.Cu at (13.6, 1.62)
- added C23: 10u, Capacitor_SMD:C_1210_3225Metric, F.Cu at (13.6, 5.88)
- added C24: 10u, Capacitor_SMD:C_1210_3225Metric, F.Cu at (29.8, 1.62)
- added C25: 47n, Capacitor_SMD:C_0402_1005Metric, F.Cu at (3.85, 15.2)
- added C26: 1u, Capacitor_SMD:C_0402_1005Metric, F.Cu at (25.5, 0.48)
- added C27: 1u, Capacitor_SMD:C_0402_1005Metric, F.Cu at (3.85, 17.2)
- added C28: 10u, Capacitor_SMD:C_1210_3225Metric, F.Cu at (13.6, 10.1)
- added C29: 1u, Capacitor_SMD:C_0402_1005Metric, F.Cu at (27.8, 22.2)
- added C30: 1u, Capacitor_SMD:C_0402_1005Metric, F.Cu at (20.0, 15.2)
- added C31: 10u, Capacitor_SMD:C_1210_3225Metric, F.Cu at (19.3, 1.62)
- added C32: 10u, Capacitor_SMD:C_1210_3225Metric, F.Cu at (19.3, 5.88)
- added C33: 10u, Capacitor_SMD:C_1210_3225Metric, F.Cu at (19.3, 10.1)
- added C34: 100n, Capacitor_SMD:C_0402_1005Metric, F.Cu at (3.85, 19.2)
- added C35: 100n, Capacitor_SMD:C_0402_1005Metric, F.Cu at (25.5, 2.46)
- added C36: 100n, Capacitor_SMD:C_0402_1005Metric, F.Cu at (3.85, 21.1)
- added C42: 100n, Capacitor_SMD:C_0402_1005Metric, F.Cu at (32.7, 30.1)
- added C43: 100n, Capacitor_SMD:C_0402_1005Metric, F.Cu at (0.94, 33.7)
- added C44: 100n, Capacitor_SMD:C_0402_1005Metric, F.Cu at (27.8, 24.2)
- added C45: 100n, Capacitor_SMD:C_0402_1005Metric, F.Cu at (25.5, 4.42)
- added C46: 100n, Capacitor_SMD:C_0402_1005Metric, F.Cu at (20.0, 17.2)
- added C47: 100n, Capacitor_SMD:C_0402_1005Metric, F.Cu at (20.0, 19.2)
- added C48: 100n, Capacitor_SMD:C_0402_1005Metric, F.Cu at (20.0, 21.1)
- added C49: 100n, Capacitor_SMD:C_0402_1005Metric, F.Cu at (20.0, 23.1)
- added C50: 100n, Capacitor_SMD:C_0402_1005Metric, F.Cu at (20.0, 25.1)
- added C51: 100n, Capacitor_SMD:C_0402_1005Metric, F.Cu at (20.0, 27.1)
- added C52: 100n, Capacitor_SMD:C_0402_1005Metric, F.Cu at (5.80, 33.7)
- added C53: 100n, Capacitor_SMD:C_0402_1005Metric, F.Cu at (27.8, 32.1)
- added C54: 100n, Capacitor_SMD:C_0402_1005Metric, F.Cu at (3.85, 23.1)
- added C55: 100n, Capacitor_SMD:C_0402_1005Metric, F.Cu at (3.85, 25.1)
- added C56: 100n, Capacitor_SMD:C_0402_1005Metric, F.Cu at (27.8, 26.1)
- added C6: 47u, Resistor_SMD:R_1210_3225Metric, F.Cu at (13.7, 16.4)
- added C7: 10u, Capacitor_SMD:C_1210_3225Metric, F.Cu at (8.11, 16.4)
- added C73: 1n, Capacitor_SMD:C_0402_1005Metric, F.Cu at (25.5, 6.39)
- added C74: 1n, Capacitor_SMD:C_0402_1005Metric, F.Cu at (25.5, 8.37)
- added C8: 10u, Capacitor_SMD:C_1210_3225Metric, F.Cu at (8.11, 20.6)
- added D4: BZT52C10, simplified_spincoater_v1:BZT52C10, F.Cu at (6.61, 24.4)
- added R11: 100k, Resistor_SMD:R_0402_1005Metric, F.Cu at (0.95, 15.2)
- added R12: 422k, Resistor_SMD:R_0402_1005Metric, F.Cu at (0.95, 17.2)
- added R13: 100k, Resistor_SMD:R_0402_1005Metric, F.Cu at (27.8, 30.1)
- added R21: 10k, Resistor_SMD:R_0402_1005Metric, F.Cu at (22.9, 15.2)
- added R23: 100r, Resistor_SMD:R_0201_0603Metric, F.Cu at (15.3, 19.3)
- added R25: 30k9, Resistor_SMD:R_0402_1005Metric, F.Cu at (0.95, 19.2)
- added R29: 2m, Resistor_SMD:R_0612_1632Metric, F.Cu at (28.3, 16.7)
- added R30: 2m, Resistor_SMD:R_0612_1632Metric, F.Cu at (32.4, 16.7)
- added R32: 22r, Resistor_SMD:R_0402_1005Metric, F.Cu at (28.4, 4.75)
- added R33: 22r, Resistor_SMD:R_0402_1005Metric, F.Cu at (28.4, 6.74)
- added R34: 10k, Resistor_SMD:R_0402_1005Metric, F.Cu at (0.95, 21.2)
- added R35: 22k1, Resistor_SMD:R_0402_1005Metric, F.Cu at (0.95, 23.2)
- added R36: 22k1, Resistor_SMD:R_0402_1005Metric, F.Cu at (0.95, 25.2)
- added R37: 10k, Resistor_SMD:R_0402_1005Metric, F.Cu at (0.95, 27.2)
- added R38: 10k, Resistor_SMD:R_0402_1005Metric, F.Cu at (30.6, 22.2)
- added TP8: TestPoint, TestPoint:TestPoint_Loop_D2.54mm_Drill1.5mm_Beaded, F.Cu at (13.7, 25.3)
- added U12: ~, simplified_spincoater_v1:XL-1005UOC, F.Cu at (12.7, 19.5)
- added U19: ~, simplified_spincoater_v1:XL-1005UOC, F.Cu at (12.7, 21.5)
- added U5: ~, simplified_spincoater_v1:AON7409, F.Cu at (8.34, 28.6)
- C5: footprint Capacitor_SMD:C_0402_1005Metric -> Resistor_SMD:R_1210_3225Metric
- R17, R31: footprint Resistor_SMD:R_0201_0603Metric -> Resistor_SMD:R_0402_1005Metric
- R22: value 30k9 -> 100r
- R28: value 22r -> 2m; footprint Resistor_SMD:R_0201_0603Metric -> Resistor_SMD:R_0612_1632Metric
- moved U4 223.4 mm to (276.0, 100.9), turned to 90 degrees
- moved D4 220.3 mm to (267.0, 109.6), turned to 90 degrees
- moved D3 216.8 mm to (268.1, 101.0), turned to 180 degrees
- moved R11 213.9 mm to (269.0, 109.0), turned to 90 degrees
- moved R10 213.6 mm to (269.0, 106.5), turned to 90 degrees
- moved U5 209.6 mm to (263.5, 109.3), turned to 180 degrees
- moved R9 202.4 mm to (260.4, 96.2)
- moved U1 202.4 mm to (257.2, 110.7)
- moved L2 14.3 mm to (47.5, 171.0), turned to 90 degrees
Connections:
- R22 pad 2: Net-(D9-A) -> Net-(R22-Pad2)
- R28 pad 2: /motor/Gate Driver/H_BRIDGE_SPC -> /motor/Gate Driver/H_BRIDGE_SPA
- U10 pad 1: GND -> /CAN Transceiver/CAN_TX
- U10 pad 4: unconnected-(U10-RXD-Pad4) -> /CAN Transceiver/CAN_RX
- U10 pad 6: /CANL -> /CAN Transceiver/CANL
- U10 pad 7: /CANH -> /CAN Transceiver/CANH
- U10 pad 9: /CAN Transceiver/CAN_TX -> GND
- U18 pad 1: GND -> /CAN Transceiver1/CAN_TX
- U18 pad 4: unconnected-(U18-RXD-Pad4) -> /CAN Transceiver1/CAN_RX
- U18 pad 9: /CAN Transceiver1/CAN_TX -> GND
- U4 pad A4: /USB/RAW_VBUS -> /Power/VBUS_IN

Commit message: fix
Parts:
- D4 (x2): value BZT52C10 -> D_SOD-123F
- U1: value HUSB238A-BB001-QN16R -> |HUSB238A-BB001-QN16R

Commit message: fix
Parts:
- removed C1, C10, C12, C4, C59, C9: 100n, Capacitor_SMD:C_0402_1005Metric
- removed C11: 47u, Capacitor_SMD:C_0402_1005Metric
- removed C13: 1u, Capacitor_SMD:C_0402_1005Metric
- removed the C14 at (70.2, 41.8)
- removed the C14 at (2.33, 1.62)
- removed the C15 at (2.33, 5.88)
- removed the C15 at (70.2, 43.8)
- removed the C16 at (70.2, 45.8)
- removed the C16 at (2.33, 10.1)
- removed the C17 at (7.97, 1.62)
- removed the C17 at (70.2, 47.8)
- removed the C18 at (70.2, 49.7)
- removed the C18 at (7.97, 5.88)
- removed the C19 at (7.97, 10.1)
- removed the C19 at (70.2, 51.7)
- removed C2: 10u, Capacitor_SMD:C_0402_1005Metric
- removed the C20 at (70.2, 53.7)
- removed the C20 at (13.6, 1.62)
- removed the C23 at (70.2, 61.6)
- removed the C23 at (13.6, 5.88)
- removed the C24 at (73.1, 57.6)
- removed the C24 at (29.8, 1.62)
- removed the C25 at (3.85, 15.2)
- removed the C25 at (73.1, 59.6)
- removed the C26 at (25.5, 0.48)
- removed the C26 at (73.1, 61.6)
- removed C3: 33n, Capacitor_SMD:C_0402_1005Metric
- removed the C30 at (20.0, 15.2)
- removed the C30 at (83.2, 64.2)
- removed the C31 at (19.3, 1.62)
- removed the C31 at (45.2, 52.0)
- removed the C32 at (84.7, 46.6)
- removed the C32 at (19.3, 5.88)
- removed the C34 at (3.85, 19.2)
- removed the C34 at (79.1, 22.5)
- removed the C35 at (79.1, 24.4)
- removed the C35 at (25.5, 2.46)
- removed the C36 at (79.1, 26.4)
- removed the C36 at (3.85, 21.1)
- removed C37, C38, C39, C40, C41: 4u7, Capacitor_SMD:C_0402_1005Metric
- removed the C42 at (32.7, 30.1)
- removed the C42 at (82.0, 28.4)
- removed the C43 at (82.0, 30.3)
- removed the C43 at (0.94, 33.7)
- removed the C44 at (27.8, 24.2)
- removed the C44 at (84.9, 22.5)
- removed the C45 at (84.9, 24.4)
- removed the C45 at (25.5, 4.42)
- removed the C46 at (20.0, 17.2)
- removed the C46 at (84.9, 26.4)
- removed the C47 at (84.9, 28.4)
- removed the C47 at (20.0, 19.2)
- removed the C48 at (20.0, 21.1)
- removed the C48 at (84.9, 30.3)
- removed the C49 at (87.8, 22.5)
- removed the C49 at (20.0, 23.1)
- removed the C50 at (20.0, 25.1)
- removed the C50 at (87.8, 24.4)
- removed the C51 at (20.0, 27.1)
- removed the C51 at (87.8, 26.4)
- removed the C52 at (5.80, 33.7)
- removed the C52 at (87.8, 28.4)
- removed the C53 at (27.8, 32.1)
- removed the C53 at (87.8, 30.3)
- removed the C54 at (45.2, 54.0)
- removed the C54 at (3.85, 23.1)
- removed the C55 at (3.85, 25.1)
- removed the C55 at (45.2, 55.9)
- removed the C56 at (75.9, 57.6)
- removed the C56 at (27.8, 26.1)
- removed C57: 1n, Capacitor_SMD:C_0402_1005Metric
- removed the C6 at (34.4, 154.6)
- removed the C6 at (13.7, 16.4)
- removed the C7 at (97.5, 156.6)
- removed the C7 at (8.11, 16.4)
- removed the C8 at (8.11, 20.6)
- removed the C8 at (97.5, 158.6)
- removed D10, D7, D8, D9: LED, Diode_SMD:D_0402_1005Metric
- removed the D4 at (267.0, 109.6)
- removed the D4 at (6.61, 24.4)
- removed R10: 10r, Resistor_SMD:R_0201_0603Metric
- removed the R11 at (0.95, 15.2)
- removed the R11 at (269.0, 109.0)
- removed R14, R15, R3, R6: 10k, Resistor_SMD:R_0201_0603Metric
- removed R16, R2, R23: 30k9, Resistor_SMD:R_0201_0603Metric
- removed the R21 at (48.9, 70.5)
- removed the R21 at (22.9, 15.2)
- removed R22, R23: 100r, Resistor_SMD:R_0201_0603Metric
- removed R26, R27: 22r, Resistor_SMD:R_0201_0603Metric
- removed the R29 at (78.6, 65.2)
- removed the R29 at (28.3, 16.7)
- removed the R30 at (78.6, 66.9)
- removed the R30 at (32.4, 16.7)
- removed R4, R9: 422k, Resistor_SMD:R_0201_0603Metric
- removed R5: 22k1, Resistor_SMD:R_0201_0603Metric
- removed TP5, TP6, TP7, TP8 (x2): TestPoint, TestPoint:TestPoint_Loop_D2.54mm_Drill1.5mm_Beaded
- removed the U5 at (263.5, 109.3)
- removed the U5 at (8.34, 28.6)
- added C14: 10u, Capacitor_SMD:C_1210_3225Metric, F.Cu at (2.33, 31.2)
- added C15: 10u, Capacitor_SMD:C_1210_3225Metric, F.Cu at (2.33, 35.4)
- added C16: 10u, Capacitor_SMD:C_1210_3225Metric, F.Cu at (2.33, 39.7)
- added C17: 10u, Capacitor_SMD:C_1210_3225Metric, F.Cu at (7.97, 31.2)
- added C18: 10u, Capacitor_SMD:C_1210_3225Metric, F.Cu at (7.97, 35.4)
- added C19: 10u, Capacitor_SMD:C_1210_3225Metric, F.Cu at (7.97, 39.7)
- added C20: 10u, Capacitor_SMD:C_1210_3225Metric, F.Cu at (13.6, 31.2)
- added C23: 10u, Capacitor_SMD:C_1210_3225Metric, F.Cu at (13.6, 35.4)
- added C24: 10u, Capacitor_SMD:C_1210_3225Metric, F.Cu at (50.7, 37.9)
- added C25: 47n, Capacitor_SMD:C_0402_1005Metric, B.Cu at (135.1, 104.0)
- added C26: 1u, Capacitor_SMD:C_0402_1005Metric, F.Cu at (46.4, 32.2)
- added C30: 1u, Capacitor_SMD:C_0402_1005Metric, F.Cu at (46.4, 46.0)
- added C31: 10u, Capacitor_SMD:C_1210_3225Metric, F.Cu at (19.3, 31.2)
- added C32: 10u, Capacitor_SMD:C_1210_3225Metric, F.Cu at (19.3, 35.4)
- added C34: 100n, Capacitor_SMD:C_0402_1005Metric, F.Cu at (144.0, 110.6)
- added C35: 100n, Capacitor_SMD:C_0402_1005Metric, F.Cu at (46.4, 34.1)
- added C36: 100n, Capacitor_SMD:C_0402_1005Metric, F.Cu at (131.2, 104.3)
- added C42: 100n, Capacitor_SMD:C_0402_1005Metric, F.Cu at (53.7, 5.24)
- added C43: 100n, Capacitor_SMD:C_0402_1005Metric, F.Cu at (53.7, 14.0)
- added C44: 100n, Capacitor_SMD:C_0402_1005Metric, F.Cu at (158.3, 105.3)
- added C45: 100n, Capacitor_SMD:C_0402_1005Metric, F.Cu at (46.4, 36.1)
- added C46: 100n, Capacitor_SMD:C_0402_1005Metric, F.Cu at (46.4, 48.0)
- added C47: 100n, Capacitor_SMD:C_0402_1005Metric, F.Cu at (46.4, 49.9)
- added C48: 100n, Capacitor_SMD:C_0402_1005Metric, F.Cu at (46.4, 51.9)
- added C49: 100n, Capacitor_SMD:C_0402_1005Metric, F.Cu at (46.4, 53.9)
- added C50: 100n, Capacitor_SMD:C_0402_1005Metric, F.Cu at (46.4, 55.8)
- added C51: 100n, Capacitor_SMD:C_0402_1005Metric, F.Cu at (46.4, 57.8)
- added C52: 100n, Capacitor_SMD:C_0402_1005Metric, F.Cu at (14.6, 51.3)
- added C53: 100n, Capacitor_SMD:C_0402_1005Metric, F.Cu at (125.9, 113.2)
- added C54: 100n, Capacitor_SMD:C_0402_1005Metric, B.Cu at (134.0, 105.5)
- added C55: 100n, Capacitor_SMD:C_0402_1005Metric, F.Cu at (151.8, 111.3)
- added C56: 100n, Capacitor_SMD:C_0402_1005Metric, F.Cu at (160.7, 106.3)
- added C6: 47u, Resistor_SMD:R_1210_3225Metric, F.Cu at (138.0, 95.0)
- added C7: 10u, Capacitor_SMD:C_1210_3225Metric, F.Cu at (141.7, 111.2)
- added C8: 10u, Capacitor_SMD:C_1210_3225Metric, F.Cu at (129.0, 104.6)
- added D4: BZT52C10, simplified_spincoater_v1:BZT52C10, B.Cu at (122.8, 107.4)
- added R11: 100k, Resistor_SMD:R_0402_1005Metric, B.Cu at (123.0, 110.0)
- added R21: 10k, Resistor_SMD:R_0402_1005Metric, F.Cu at (49.3, 57.1)
- added R29: 2m, Resistor_SMD:R_0612_1632Metric, F.Cu at (36.9, 29.7)
- added R30: 2m, Resistor_SMD:R_0612_1632Metric, F.Cu at (41.0, 29.7)
- added R39: 10k, Resistor_SMD:R_0402_1005Metric, F.Cu at (157.1, 96.8)
- added REF**: MountingHole_2.2mm_M2_DIN965_Pad, MountingHole:MountingHole_2.2mm_M2_DIN965_Pad, F.Cu at (158.0, 112.0)
- added S1: TS-1088-AR02016, simplified_spincoater_v1:TS-1088-AR02016, F.Cu at (158.4, 93.9)
- added S2: TS-1088-AR02016, simplified_spincoater_v1:TS-1088-AR02016, F.Cu at (148.5, 93.9)
- added U20: ~, simplified_spincoater_v1:XL-1005UOC, F.Cu at (41.0, 12.9)
- added U21: ~, simplified_spincoater_v1:XL-1005UOC, F.Cu at (41.0, 14.9)
- added U5: ~, simplified_spincoater_v1:AON7409, F.Cu at (124.5, 106.8)
- C27, D3, R25, R34, R36, U6: moved to B.Cu
- U1: value |HUSB238A-BB001-QN16R -> HUSB238A-BB001-QN16R
- moved R12 179.5 mm to (153.8, 111.3), turned to -90 degrees
- moved R35 175.5 mm to (152.8, 111.3), turned to 90 degrees
- moved R37 171.4 mm to (157.1, 97.8)
- moved U4 160.2 mm to (116.0, 108.4), turned to -90 degrees
- moved R25 159.1 mm to (133.3, 107.6), turned to 90 degrees
- moved R34 157.2 mm to (132.3, 107.6), turned to -90 degrees
- moved C29 156.8 mm to (160.7, 105.3)
- moved R38 152.9 mm to (158.3, 106.3)
- moved C27 150.5 mm to (123.0, 109.0)
- moved R36 149.8 mm to (124.9, 109.3)
- moved D3 145.6 mm to (122.9, 112.0)
- moved R13 131.0 mm to (129.0, 113.2)
- moved U1 130.3 mm to (126.9, 110.6)
- moved U6 129.2 mm to (156.1, 99.0), turned to 90 degrees
- moved C5 120.1 mm to (136.6, 104.1), turned to 90 degrees
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Connections:
- D3 pad 1: /MCU/USB_D+ -> Net-(U1-CC1)
- D3 pad 10: unconnected-(D3-Pad10) -> Net-(U1-CC1)
- D3 pad 2: /MCU/USB_D- -> Net-(U1-CC2)
- D3 pad 4: Net-(U1-CC2) -> /MCU/USB_D+
- D3 pad 5: Net-(U1-CC1) -> /MCU/USB_D-
- D3 pad 6: unconnected-(D3-Pad6) -> /MCU/USB_D-
- D3 pad 7: unconnected-(D3-Pad7) -> /MCU/USB_D+
- D3 pad 9: unconnected-(D3-Pad9) -> Net-(U1-CC2)
- U12 pad 2: Net-(R22-Pad2) -> unconnected-(U12-Pad2)
- U19 pad 2: Net-(R23-Pad2) -> unconnected-(U19-Pad2)
- U6 pad 15: unconnected-(U6-IO3-Pad15) -> /MCU/PD_INT_N
- U6 pad 16: /CAN Transceiver1/CAN_TX -> /MCU/PD_FAULT
- U6 pad 23: /MCU/PD_INT_N -> unconnected-(U6-IO21-Pad23)
- U6 pad 27: unconnected-(U6-IO0-Pad27) -> Net-(U6-IO0)
- U6 pad 28: /MCU/PD_FAULT -> unconnected-(U6-IO35-Pad28)
- U6 pad 33: /MCU/EN_12V -> unconnected-(U6-IO40-Pad33)
- U6 pad 35: unconnected-(U6-IO42-Pad35) -> /CAN Transceiver1/CAN_TX
- U6 pad 8: unconnected-(U6-IO15-Pad8) -> /MCU/EN_12V
Routing:
- net /MCU/USB_D-: track 0.00 -> 47.4 mm, vias 0 -> 2
- net /MCU/USB_D+: track 0.00 -> 44.3 mm, vias 0 -> 2
- net /MCU/EN_12V: track 0.00 -> 23.7 mm, vias 0 -> 2
- net /MCU/PD_FAULT: track 0.00 -> 22.5 mm, vias 0 -> 1
- net /MCU/PD_SDA: track 0.00 -> 22.1 mm, vias 0 -> 1
- net /MCU/PD_SCL: track 0.00 -> 20.8 mm, vias 0 -> 1
- net /MCU/PD_INT_N: track 0.00 -> 20.0 mm, vias 0 -> 1
- net Net-(U6-IO0): track 0.00 -> 16.8 mm, vias 0 -> 1
- net Net-(U2-FB): track 0.00 -> 16.5 mm, vias 0 -> 1
- net Net-(U6-EN): track 0.00 -> 14.6 mm, vias 0 -> 1
- net GND: track 0.00 -> 11.1 mm, vias 0 -> 176
- net Net-(U1-CC1): track 0.00 -> 9.07 mm, vias 0 -> 2
- net Net-(U2-SW): track 0.00 -> 8.37 mm
- net Net-(D4-A): track 0.00 -> 7.14 mm, vias 0 -> 1
- net Net-(U1-CC2): track 0.00 -> 5.96 mm, vias 0 -> 2
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- added copper zone on F.Cu, net +3V3
- added copper zone on F.Cu, net /Power/VBUS_IN
- added copper zone on F.Cu, net GND
- added copper zone on F.Cu, net Net-(U2-SW)
- added copper zone on F.Cu, net Net-(U3-SW)
- added copper zone on F.Cu, net VBUS
Other:
- board outline added: 49.7 x 49.6 mm
- copper layers 2 -> 6
- rule pad_to_mask_clearance: 0 -> 0.038

Commit message: fix
Parts:
- C21, C26, C30, C45, C46, C47, C48, C49, C50, C51, C55, R12, R35: moved to B.Cu
- moved C43 139.9 mm to (165.9, 97.5)
- moved U18 139.5 mm to (162.2, 91.8)
- moved U11 138.8 mm to (155.5, 85.0)
- moved U10 137.5 mm to (162.5, 96.9)
- moved C42 136.5 mm to (158.5, 92.7)
- moved U13 133.0 mm to (151.4, 85.0)
- moved R28 127.5 mm to (147.8, 85.0)
- moved U14 121.6 mm to (141.2, 84.9)
- moved C22 118.4 mm to (143.4, 98.1)
- moved C21 116.7 mm to (140.8, 96.9), turned to -90 degrees
- moved U15 115.9 mm to (137.1, 84.9)
- moved C35 113.7 mm to (142.5, 95.0), turned to 90 degrees
- moved C26 111.3 mm to (136.6, 97.5), turned to 90 degrees
- moved R29 111.2 mm to (133.5, 84.9)
- moved C24 109.3 mm to (144.7, 93.6), turned to -90 degrees
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Connections:
- net /motor/Gate Driver/GATE_DRIVER_NFALUT renamed /motor/Gate Driver/GATE_DRIVER_NFAULT
- U6 pad 41_1: (no net) -> GND
- U6 pad 41_2: (no net) -> GND
- U6 pad 41_3: (no net) -> GND
- U6 pad 41_4: (no net) -> GND
- U6 pad 41_5: (no net) -> GND
- U6 pad 41_6: (no net) -> GND
- U6 pad 41_7: (no net) -> GND
- U6 pad 41_8: (no net) -> GND
- U6 pad 41_9: (no net) -> GND
Routing:
- net Net-(U6-IO0): track 16.8 -> 35.6 mm, vias 1 -> 3
- net +12V: track 0.00 -> 12.1 mm, vias 1 -> 2
- net Net-(U6-EN): track 14.6 -> 2.63 mm
- net +3V3: track 4.84 -> 11.9 mm, vias 32 -> 40
- net Net-(U2-FB): track 16.5 -> 9.53 mm
- net Net-(U2-CB): track 5.08 -> 0.15 mm, vias 0 -> 1
- net /motor/Gate Driver/GATE_DRIVER_INLA: track 0.00 -> 2.52 mm, vias 0 -> 3
- net Net-(U8-DVDD): track 0.00 -> 2.13 mm, vias 0 -> 5
- net Net-(U2-SW): track 8.37 -> 6.39 mm, vias 0 -> 1
- net Net-(U8-CPL): track 0.00 -> 1.74 mm, vias 0 -> 1
- net /MCU/EN_12V: track 23.7 -> 22.0 mm, vias 2 -> 3
- net Net-(U8-CPH): track 0.00 -> 1.69 mm, vias 0 -> 1
- net /MCU/PD_FAULT: track 22.5 -> 21.1 mm, vias 1 -> 2
- net /MCU/PD_SCL: track 20.8 -> 19.4 mm
- net /MCU/PD_SDA: track 22.1 -> 20.8 mm
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- added copper zone on In1.Cu, net GND
- added copper zone on In4.Cu, net GND
- added copper zone on B.Cu, net Net-(U8-DVDD)
- added copper zone on F.Cu, net Net-(U8-DVDD)
Other:
- board size 49.7 x 49.6 mm -> 49.7 x 49.8 mm
