File: electronics/simplified/v1/simplified_spincoater_v1/simplified_spincoater_v1.kicad_sch (KiCad schematic)
At the start: 0 parts

Commit message: fix
Changed lines of the file:
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@@
 	(wire
 		(pts
-			(xy 220.98 99.06) (xy 231.14 99.06)
+			(xy 220.98 99.06) (xy 228.6 99.06)
 		)
 		(stroke
@@
 	(wire
 		(pts
-			(xy 137.16 91.44) (xy 231.14 91.44)
-		)
-		(stroke
-			(width 0)
-			(type default)
-		)
-	)
-	(wire
-		(pts
-			(xy 220.98 101.6) (xy 231.14 101.6)
+			(xy 137.16 91.44) (xy 228.6 91.44)
+		)
+		(stroke
+			(width 0)
+			(type default)
+		)
+	)
+	(wire
+		(pts
+			(xy 220.98 101.6) (xy 228.6 101.6)
 		)
 		(stroke
@@
 	(sheet
 		(at 147.32 96.52)
-		(size 30.48 7.62)
+		(size 33.02 7.62)
 		(exclude_from_sim no)
 		(in_bom yes)
@@
 		)
 		(pin "CANH" bidirectional
-			(at 177.8 99.06 0)
+			(at 180.34 99.06 0)
 			(effects
 				(font
@@
 		)
 		(pin "CANL" bidirectional
-			(at 177.8 101.6 0)
+			(at 180.34 101.6 0)
 			(effects
 				(font
@@
 	)
 	(sheet
-		(at 231.14 88.9)
+		(at 228.6 88.9)
 		(size 22.86 15.24)
 		(exclude_from_sim no)
@@
 		)
 		(property "Sheetname" "motor"
-			(at 231.14 88.1884 0)
+			(at 228.6 88.1884 0)
 			(effects
 				(font
@@
 		)
 		(property "Sheetfile" "motor.kicad_sch"
-			(at 231.14 104.7246 0)
+			(at 228.6 104.7246 0)
 			(effects
 				(font
@@
 		)
 		(pin "STM32_EN" input
-			(at 231.14 91.44 180)
+			(at 228.6 91.44 180)
 			(effects
 				(font
@@
 		)
 		(pin "CAN_RX" input
-			(at 231.14 99.06 180)
+			(at 228.6 99.06 180)
 			(effects
 				(font
@@
 		)
 		(pin "CAN_TX" input
-			(at 231.14 101.6 180)
-			(effects
-				(font
+			(at 228.6 101.6 180)
+			(effects
+				(font

Commit message: fix
Parts:
- added J2: Conn_01x30_Socket, symbol Connector:Conn_01x30_Socket
