File: electronics/main_board/main_board.kicad_pcb (KiCad board)
At the start: 6 copper layers, 49.7 x 49.8 mm, 91 parts, among them U1 HUSB238A-BB001-QN16R, U10 TJA1051TK/3, U11 NTTFS5C454NL, U13 NTTFS5C454NL, U14 NTTFS5C454NL, U15 NTTFS5C454NL, U16 NTTFS5C454NL, U17 NTTFS5C454NL, U18 TJA1051TK/3, U2 LMR51420YDD, U3 TPS62933DRL, U4 GT-USB-7004N, U6 ESP32-S3-WROOM-1, U7 STM32G474VEH6, U8 DRV8323SRTA, U9 AS5600

Commit message: fix
Parts:
- removed C52: 100n, Capacitor_SMD:C_0402_1005Metric
- added ?: , , F.Cu at (104.0, 101.0)
- added ?: , , F.Cu at (115.6, 111.6)
- D4: value BZT52C10 -> D_SOD-123F
- U9: value AS5600 -> val; footprint main_board:AS5600 -> main_board:AFD01-S35FCA-00
- moved U9 53.6 mm to (126.8, 76.6)
- moved C47 20.3 mm to (148.8, 91.0)
- moved C49 20.3 mm to (150.0, 93.8)
- moved C50 20.3 mm to (145.6, 91.0)
- moved U7 20.3 mm to (147.6, 93.4)
- moved C30 20.3 mm to (148.5, 97.1)
- moved C46 20.3 mm to (147.2, 91.0)
- moved C48 20.3 mm to (146.0, 93.8)
- moved C51 20.3 mm to (148.5, 96.2)
- moved C21 20.2 mm to (120.7, 95.8)
- moved C26 20.2 mm to (116.4, 96.4)
- moved C35 20.2 mm to (122.3, 94.0)
- moved C45 20.2 mm to (115.0, 93.7)
- moved U8 20.2 mm to (117.8, 93.9)
- moved C22 20.2 mm to (123.2, 97.0)
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Connections:
- net /motor/Gate Driver/GATE_DRIVER_ENABLE renamed /Motor/Gate Driver/GATE_DRIVER_ENABLE
- net /motor/Gate Driver/GATE_DRIVER_INHA renamed /Motor/Gate Driver/GATE_DRIVER_INHA
- net /motor/Gate Driver/GATE_DRIVER_INHB renamed /Motor/Gate Driver/GATE_DRIVER_INHB
- net /motor/Gate Driver/GATE_DRIVER_INHC renamed /Motor/Gate Driver/GATE_DRIVER_INHC
- net /motor/Gate Driver/GATE_DRIVER_INLA renamed /Motor/Gate Driver/GATE_DRIVER_INLA
- net /motor/Gate Driver/GATE_DRIVER_NFAULT renamed /Motor/Gate Driver/GATE_DRIVER_NFAULT
- net /motor/Gate Driver/GATE_DRIVER_NSCS renamed /Motor/Gate Driver/GATE_DRIVER_NSCS
- net /motor/Gate Driver/GATE_DRIVER_SCLK renamed /Motor/Gate Driver/GATE_DRIVER_SCLK
- net /motor/Gate Driver/GATE_DRIVER_SDI renamed /Motor/Gate Driver/GATE_DRIVER_SDI
- net /motor/Gate Driver/GATE_DRIVER_SDO renamed /Motor/Gate Driver/GATE_DRIVER_SDO
- net /motor/Gate Driver/H_BRIDGE_GHA renamed /Motor/Gate Driver/H_BRIDGE_GHA
- net /motor/Gate Driver/H_BRIDGE_GHB renamed /Motor/Gate Driver/H_BRIDGE_GHB
- net /motor/Gate Driver/H_BRIDGE_GHC renamed /Motor/Gate Driver/H_BRIDGE_GHC
- net /motor/Gate Driver/H_BRIDGE_GLA renamed /Motor/Gate Driver/H_BRIDGE_GLA
- net /motor/Gate Driver/H_BRIDGE_GLB renamed /Motor/Gate Driver/H_BRIDGE_GLB
- net /motor/Gate Driver/H_BRIDGE_GLC renamed /Motor/Gate Driver/H_BRIDGE_GLC
- net /motor/Gate Driver/H_BRIDGE_SPA renamed /Motor/Gate Driver/H_BRIDGE_SPA
- net /motor/Gate Driver/H_BRIDGE_SPB renamed /Motor/Gate Driver/H_BRIDGE_SPB
- net /motor/Gate Driver/H_BRIDGE_SPC renamed /Motor/Gate Driver/H_BRIDGE_SPC
- net /motor/Gate Driver/MOTOR_A_CURRENT_SENSE renamed /Motor/Gate Driver/MOTOR_A_CURRENT_SENSE
- net /motor/Gate Driver/MOTOR_B_CURRENT_SENSE renamed /Motor/Gate Driver/MOTOR_B_CURRENT_SENSE
- net /motor/Gate Driver/MOTOR_C_CURRENT_SENSE renamed /Motor/Gate Driver/MOTOR_C_CURRENT_SENSE
- U10 pad 6: /CAN Transceiver/CANL -> /CANL
- U10 pad 7: /CAN Transceiver/CANH -> /CANH
- U11 pad 1: /motor/H-Bridge/MOTOR_A -> /Motor/H-Bridge/MOTOR_A
- U11 pad 2: /motor/H-Bridge/MOTOR_A -> /Motor/H-Bridge/MOTOR_A
- U11 pad 3: /motor/H-Bridge/MOTOR_A -> /Motor/H-Bridge/MOTOR_A
- U13 pad 5: /motor/H-Bridge/MOTOR_A -> /Motor/H-Bridge/MOTOR_A
- U13 pad 6: /motor/H-Bridge/MOTOR_A -> /Motor/H-Bridge/MOTOR_A
- U13 pad 7: /motor/H-Bridge/MOTOR_A -> /Motor/H-Bridge/MOTOR_A
- U13 pad 8: /motor/H-Bridge/MOTOR_A -> /Motor/H-Bridge/MOTOR_A
- U14 pad 1: /motor/H-Bridge/MOTOR_B -> /Motor/H-Bridge/MOTOR_B
- U14 pad 2: /motor/H-Bridge/MOTOR_B -> /Motor/H-Bridge/MOTOR_B
- U14 pad 3: /motor/H-Bridge/MOTOR_B -> /Motor/H-Bridge/MOTOR_B
- U15 pad 5: /motor/H-Bridge/MOTOR_B -> /Motor/H-Bridge/MOTOR_B
- U15 pad 6: /motor/H-Bridge/MOTOR_B -> /Motor/H-Bridge/MOTOR_B
- U15 pad 7: /motor/H-Bridge/MOTOR_B -> /Motor/H-Bridge/MOTOR_B
- U15 pad 8: /motor/H-Bridge/MOTOR_B -> /Motor/H-Bridge/MOTOR_B
- U16 pad 1: /motor/H-Bridge/MOTOR_C -> /Motor/H-Bridge/MOTOR_C
- U16 pad 2: /motor/H-Bridge/MOTOR_C -> /Motor/H-Bridge/MOTOR_C
- U16 pad 3: /motor/H-Bridge/MOTOR_C -> /Motor/H-Bridge/MOTOR_C
- U17 pad 5: /motor/H-Bridge/MOTOR_C -> /Motor/H-Bridge/MOTOR_C
- U17 pad 6: /motor/H-Bridge/MOTOR_C -> /Motor/H-Bridge/MOTOR_C
- U17 pad 7: /motor/H-Bridge/MOTOR_C -> /Motor/H-Bridge/MOTOR_C
- U17 pad 8: /motor/H-Bridge/MOTOR_C -> /Motor/H-Bridge/MOTOR_C
- U6 pad 12: unconnected-(U6-IO8-Pad12) -> /Expansion Port/EXPANSION_IO8
- U6 pad 15: /MCU/PD_INT_N -> /Expansion Port/EXPANSION_IO3
- U6 pad 16: /MCU/PD_FAULT -> /Expansion Port/EXPANSION_IO46
- U6 pad 17: unconnected-(U6-IO9-Pad17) -> /Expansion Port/EXPANSION_IO9
- U6 pad 18: unconnected-(U6-IO10-Pad18) -> /Expansion Port/EXPANSION_IO10
- U6 pad 19: unconnected-(U6-IO11-Pad19) -> /Expansion Port/EXPANSION_IO11
- U6 pad 20: unconnected-(U6-IO12-Pad20) -> /Expansion Port/EXPANSION_IO12
- U6 pad 21: unconnected-(U6-IO13-Pad21) -> /Expansion Port/EXPANSION_IO13
- U6 pad 22: unconnected-(U6-IO14-Pad22) -> /Expansion Port/EXPANSION_IO14
- U6 pad 23: unconnected-(U6-IO21-Pad23) -> /Expansion Port/EXPANSION_IO21
- U6 pad 24: unconnected-(U6-IO47-Pad24) -> /Expansion Port/EXPANSION_IO47
- U6 pad 25: unconnected-(U6-IO48-Pad25) -> /Expansion Port/EXPANSION_IO48
- U6 pad 26: /CAN Transceiver1/CAN_RX -> /Expansion Port/EXPANSION_IO45
- U6 pad 28: unconnected-(U6-IO35-Pad28) -> /Expansion Port/EXPANSION_IO35
- U6 pad 29: unconnected-(U6-IO36-Pad29) -> /Expansion Port/EXPANSION_IO36
- U6 pad 30: unconnected-(U6-IO37-Pad30) -> /Expansion Port/EXPANSION_IO37
- U6 pad 31: unconnected-(U6-IO38-Pad31) -> /Expansion Port/EXPANSION_IO38
- U6 pad 33: unconnected-(U6-IO40-Pad33) -> /Expansion Port/EXPANSION_IO40
- U6 pad 34: unconnected-(U6-IO41-Pad34) -> /Expansion Port/EXPANSION_IO41
- U6 pad 35: /CAN Transceiver1/CAN_TX -> /Expansion Port/EXPANSION_IO42
- U6 pad 38: unconnected-(U6-IO2-Pad38) -> /Expansion Port/EXPANSION_IO2
- U6 pad 39: unconnected-(U6-IO1-Pad39) -> /Expansion Port/EXPANSION_IO1
- U6 pad 4: unconnected-(U6-IO4-Pad4) -> /MCU/EN_12V
- U6 pad 5: unconnected-(U6-IO5-Pad5) -> /MCU/PD_INT_N
- U6 pad 6: unconnected-(U6-IO6-Pad6) -> /MCU/PD_FAULT
- U6 pad 7: unconnected-(U6-IO7-Pad7) -> /CAN Transceiver1/CAN_RX
- U6 pad 8: /MCU/EN_12V -> /CAN Transceiver1/CAN_TX
- U6 pad 9: unconnected-(U6-IO16-Pad9) -> /Expansion Port/EXPANSION_IO16
- U7 pad C10: /motor/Encoder/ENCODER_SCL -> /Expansion Port/ENCODER_SCL
- U7 pad D9: /motor/Encoder/ENCODER_SDA -> /Expansion Port/ENCODER_SDA
- U8 pad 14: /motor/H-Bridge/MOTOR_B -> /Motor/H-Bridge/MOTOR_B
- U8 pad 17: /motor/H-Bridge/MOTOR_C -> /Motor/H-Bridge/MOTOR_C
- U8 pad 7: /motor/H-Bridge/MOTOR_A -> /Motor/H-Bridge/MOTOR_A
- U9 pad 1: +3V3 -> unconnected-(U9-Pad1)
- U9 pad 2: +3V3 -> unconnected-(U9-Pad2)
- U9 pad 4: GND -> unconnected-(U9-Pad4)
- U9 pad 6: /motor/Encoder/ENCODER_SDA -> unconnected-(U9-Pad6)
- U9 pad 7: /motor/Encoder/ENCODER_SCL -> unconnected-(U9-Pad7)
Routing:
- net /MCU/PD_INT_N: track 19.9 -> 30.7 mm
- net /MCU/PD_FAULT: track 21.1 -> 29.8 mm
- net /MCU/EN_12V: track 22.0 -> 20.8 mm
- net Net-(U2-SW): track 6.39 -> 7.43 mm
- net /motor/H-Bridge/MOTOR_C: track 0.98 -> 0.00 mm, vias 1 -> 0
- net /Motor/H-Bridge/MOTOR_C: track 0.00 -> 0.98 mm, vias 0 -> 1
- net /motor/H-Bridge/MOTOR_B: track 0.96 -> 0.00 mm, vias 1 -> 0
- net /Motor/H-Bridge/MOTOR_B: track 0.00 -> 0.96 mm, vias 0 -> 1
- net /motor/H-Bridge/MOTOR_A: track 0.88 -> 0.00 mm, vias 1 -> 0
- net /Motor/H-Bridge/MOTOR_A: track 0.00 -> 0.88 mm, vias 0 -> 1
- net /MCU/PD_SCL: track 19.4 -> 18.7 mm
- net /MCU/PD_SDA: track 20.8 -> 20.2 mm
- net Net-(U6-IO0): track 35.6 -> 35.1 mm
- net VBUS: vias 123 -> 132
- net (no net): vias 15 -> 39

Commit message: fix
Parts:
- removed ? (x2): , 
- removed the REF** at (160.0, 112.0)
- added REF**: MountingHole_2.2mm_M2_DIN965_Pad, MountingHole:MountingHole_2.2mm_M2_DIN965_Pad, F.Cu at (160.5, 112.2)
- added REF**: MountingHole_2.2mm_M2_DIN965_Pad, MountingHole:MountingHole_2.2mm_M2_DIN965_Pad, F.Cu at (117.0, 112.0)
- D4: value D_SOD-123F -> BZT52C10
- U9: value val -> AFD01-S35FCA-00
- moved C21 6.53 mm to (127.2, 95.8)
- moved C26 6.53 mm to (122.9, 96.4)
- moved C35 6.53 mm to (128.8, 94.0)
- moved C45 6.53 mm to (121.5, 93.7)
- moved U8 6.53 mm to (124.3, 93.9)
- moved C22 6.53 mm to (129.8, 97.0)
- moved C24 6.53 mm to (131.1, 92.6)
- moved U4 0.71 mm to (116.0, 104.7)
- moved R36 0.37 mm to (125.3, 109.3)
- moved C27 0.30 mm to (123.3, 109.0)
- moved R11 0.30 mm to (123.3, 110.0)
Routing:
- net Net-(U1-CC2): track 5.96 -> 11.8 mm, vias 2 -> 3
- net +12V: track 12.1 -> 7.14 mm, vias 2 -> 21
- net Net-(U1-CC1): track 9.07 -> 14.0 mm
- net /MCU/USB_D+: track 44.2 -> 47.9 mm
- net /MCU/USB_D-: track 47.3 -> 51.0 mm
- net /Power/VBUS_IN: track 3.99 -> 2.70 mm, vias 1 -> 0
- net VBUS: vias 132 -> 131
- net GND: vias 229 -> 197
- net +3V3: vias 40 -> 45
- added copper zone on F.Cu, net +12V

Commit message: fix
Parts:
- removed U4: GT-USB-7004N, main_board:GT-USB-7004N
- added USB1: GT-USB-7004N, main_board:GT-USB-7004N, F.Cu at (117.7, 104.4)
- moved U5 0.74 mm to (123.7, 106.8)
Routing:
- net Net-(D4-A): track 7.08 -> 7.96 mm
- net VBUS: vias 131 -> 133

Commit message: fix
Parts:
- removed the REF** at (160.5, 112.2)
- added CN1: DB141R-2.54-2P, main_board:DB141R-2.54-2P-GN, F.Cu at (157.5, 85.0)
- added CN3: KF202-5.0-3P, main_board:KF202-5.0-3P, F.Cu at (147.3, 74.6)
- added REF**: MountingHole_2.2mm_M2_DIN965_Pad, MountingHole:MountingHole_2.2mm_M2_DIN965_Pad, F.Cu at (161.0, 76.0)
- added REF**: MountingHole_2.2mm_M2_DIN965_Pad, MountingHole:MountingHole_2.2mm_M2_DIN965_Pad, F.Cu at (161.0, 112.0)
- added REF**: MountingHole_2.2mm_M2_DIN965_Pad, MountingHole:MountingHole_2.2mm_M2_DIN965_Pad, F.Cu at (117.0, 81.0)
- C45: moved to F.Cu
- C58, C73, C74, R17, R21, R31, R32, R33: moved to B.Cu
- moved C43 46.8 mm to (119.5, 91.7), turned to 90 degrees
- moved C58 45.2 mm to (136.7, 96.8), turned to 45 degrees
- moved U10 43.7 mm to (118.9, 95.1), turned to 90 degrees
- moved C73 43.6 mm to (135.8, 95.8), turned to 45 degrees
- moved C74 42.3 mm to (134.9, 94.9), turned to 45 degrees
- moved C42 39.1 mm to (197.5, 96.0)
- moved U18 39.1 mm to (201.1, 95.2)
- moved R31 37.5 mm to (135.3, 98.1), turned to -135 degrees
- moved R32 35.1 mm to (134.4, 97.2), turned to -135 degrees
- moved R17 33.4 mm to (132.3, 93.4), turned to -90 degrees
- moved R33 32.9 mm to (133.6, 96.2), turned to -135 degrees
- moved R21 32.6 mm to (128.3, 98.7), turned to -90 degrees
- moved C47 22.1 mm to (127.0, 94.2), turned to 180 degrees
- moved C49 21.1 mm to (129.0, 93.7), turned to 90 degrees
- moved C46 21.0 mm to (127.0, 96.6), turned to 180 degrees
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Connections:
- net /Motor/H-Bridge/MOTOR_A renamed /Motor/Gate Driver/H_BRIDGE_SHA
- net /Motor/H-Bridge/MOTOR_B renamed /Motor/Gate Driver/H_BRIDGE_SHB
- net /Motor/H-Bridge/MOTOR_C renamed /Motor/Gate Driver/H_BRIDGE_SHC
Routing:
- net Net-(U6-IO0): track 35.1 -> 3.94 mm, vias 3 -> 1
- net /Motor/Gate Driver/GATE_DRIVER_INLA: track 2.52 -> 24.9 mm, vias 3 -> 2
- net /Motor/Gate Driver/GATE_DRIVER_INHB: track 0.84 -> 17.5 mm, vias 1 -> 2
- net /Motor/Gate Driver/GATE_DRIVER_INHA: track 0.83 -> 17.1 mm, vias 1 -> 2
- net /Motor/Gate Driver/GATE_DRIVER_INHC: track 0.84 -> 16.8 mm, vias 1 -> 2
- net /MCU/EN_12V: track 20.8 -> 4.92 mm, vias 3 -> 2
- net /Motor/Gate Driver/GATE_DRIVER_SDO: track 0.91 -> 15.7 mm, vias 1 -> 2
- net /Motor/Gate Driver/GATE_DRIVER_SCLK: track 0.92 -> 14.3 mm, vias 1 -> 2
- net /Motor/Gate Driver/GATE_DRIVER_ENABLE: track 0.93 -> 13.6 mm
- net /Motor/Gate Driver/GATE_DRIVER_SDI: track 0.92 -> 12.6 mm, vias 1 -> 2
- net /Motor/Gate Driver/GATE_DRIVER_NFAULT: track 0.91 -> 10.3 mm
- net /Motor/Gate Driver/GATE_DRIVER_NSCS: track 0.92 -> 9.58 mm, vias 1 -> 2
- net +12V: track 7.14 -> 0.00 mm, vias 21 -> 0
- net /Motor/Gate Driver/MOTOR_A_CURRENT_SENSE: track 0.00 -> 7.00 mm, vias 0 -> 1
- net /Motor/Gate Driver/MOTOR_B_CURRENT_SENSE: track 0.00 -> 6.40 mm, vias 0 -> 1
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- removed copper zone on F.Cu, net +12V
- removed copper zone on B.Cu, net Net-(U8-DVDD)
- removed copper zone on F.Cu, net Net-(U8-DVDD)
Other:
- board size 49.7 x 49.8 mm -> 50 x 47 mm

Commit message: fix
Parts:
- added R18: 120, Resistor_SMD:R_0402_1005Metric, F.Cu at (117.0, 96.7)
- added R19: 120, Resistor_SMD:R_0402_1005Metric, F.Cu at (159.7, 97.1)
- added R40: 10k, Resistor_SMD:R_0402_1005Metric, B.Cu at (137.9, 108.7)
- added R41: 10k, Resistor_SMD:R_0402_1005Metric, B.Cu at (136.0, 108.7)
- added R42: 10k, Resistor_SMD:R_0402_1005Metric, B.Cu at (138.9, 108.7)
- added R43: 10k, Resistor_SMD:R_0402_1005Metric, B.Cu at (137.0, 108.7)
- moved U18 41.6 mm to (159.7, 99.7), turned to 90 degrees
- moved C42 38.4 mm to (159.6, 102.4), turned to 180 degrees
- moved R29 10.2 mm to (140.0, 86.0), turned to 180 degrees
- moved U14 6.85 mm to (131.5, 86.1), turned to 90 degrees
- moved C43 5.75 mm to (122.3, 96.7), turned to -90 degrees
- moved C35 3.57 mm to (145.3, 94.3)
- moved C22 3.57 mm to (146.4, 95.9)
- moved C24 3.57 mm to (148.5, 95.1)
- moved U15 2.40 mm to (136.2, 86.0), turned to 90 degrees
- moved U10 1.78 mm to (119.7, 96.7), turned to 180 degrees
Connections:
- net /CANH renamed /CAN_P
- net /CANL renamed /CAN_N
Routing:
- net /CAN_N: track 0.00 -> 58.6 mm
- net /CAN_P: track 0.00 -> 58.4 mm, vias 0 -> 2
- net GND: track 12.7 -> 63.9 mm, vias 155 -> 186
- net /Motor/Gate Driver/H_BRIDGE_SPC: track 0.00 -> 25.7 mm, vias 0 -> 2
- net /Motor/Gate Driver/H_BRIDGE_GLC: track 0.00 -> 23.1 mm, vias 0 -> 2
- net /Motor/Gate Driver/H_BRIDGE_SHC: track 0.00 -> 21.0 mm, vias 0 -> 2
- net /Motor/Gate Driver/H_BRIDGE_GHC: track 0.18 -> 17.7 mm, vias 0 -> 2
- net /MCU/EN_12V: track 4.92 -> 22.3 mm
- net VBUS: track 0.00 -> 15.2 mm, vias 133 -> 2
- net /Motor/Gate Driver/H_BRIDGE_GHA: track 0.37 -> 14.3 mm, vias 0 -> 2
- net /CAN Transceiver1/CAN_TX: track 0.00 -> 11.3 mm, vias 0 -> 1
- net /CAN Transceiver1/CAN_RX: track 0.00 -> 11.1 mm, vias 0 -> 1
- net /Motor/Gate Driver/H_BRIDGE_SHA: track 0.00 -> 10.7 mm, vias 0 -> 2
- net Net-(U6-IO0): track 3.94 -> 14.4 mm, vias 1 -> 0
- net /Motor/Gate Driver/H_BRIDGE_GHB: track 0.00 -> 10.2 mm, vias 0 -> 2
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
Commit message: fix
Parts:
- C14, C15, C17, C20, C23, C28, C31, C32, C33: moved to B.Cu
- C5, C6: footprint Resistor_SMD:R_1210_3225Metric -> Capacitor_SMD:C_1210_3225Metric
- C55, R12, R35: moved to F.Cu
- moved C14 78.5 mm to (135.3, 83.7)
- moved C33 74.1 mm to (149.1, 83.7), turned to 180 degrees
- moved C15 63.5 mm to (116.6, 97.4), turned to 180 degrees
- moved C16 60.0 mm to (116.6, 90.9), turned to 180 degrees
- moved C17 58.8 mm to (120.7, 83.7), turned to 180 degrees
- moved C18 57.1 mm to (116.6, 94.2), turned to 180 degrees
- moved C19 56.7 mm to (116.6, 97.4), turned to 180 degrees
- moved C23 50.6 mm to (116.6, 90.9), turned to 180 degrees
- moved C28 50.2 mm to (116.6, 94.1), turned to 180 degrees
- moved C20 29.2 mm to (66.1, 96.6), turned to -90 degrees
- moved C31 29.0 mm to (69.3, 96.0), turned to -90 degrees
- moved C32 24.3 mm to (72.5, 96.0), turned to -90 degrees
- moved REF** 21.2 mm to (96.0, 84.0)
- moved R18 7.06 mm to (121.7, 91.4), turned to 0 degrees
- moved U10 3.35 mm to (121.7, 94.0), turned to 90 degrees
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Routing:
- net /MCU/EN_12V: track 22.3 -> 3.97 mm
- net /CAN_N: track 58.6 -> 47.4 mm, vias 0 -> 2
- net /CAN_P: track 58.4 -> 48.6 mm, vias 2 -> 0
- net +3V3: track 14.2 -> 19.3 mm, vias 42 -> 17
- net GND: track 63.9 -> 60.5 mm
- net Net-(U8-VCP): track 0.00 -> 3.17 mm
- net Net-(U2-CB): track 0.00 -> 2.62 mm
- net /Motor/Gate Driver/H_BRIDGE_SPC: track 25.7 -> 23.6 mm
- net /CAN Transceiver/CAN_TX: track 3.92 -> 5.91 mm
- net /Motor/Gate Driver/H_BRIDGE_GLC: track 23.1 -> 21.1 mm
- net Net-(U2-FB): track 9.53 -> 7.63 mm, vias 1 -> 0
- net /Motor/Gate Driver/GATE_DRIVER_SCLK: track 16.9 -> 15.0 mm
- net VBUS: track 15.2 -> 13.4 mm, vias 2 -> 157
- net /Motor/Gate Driver/GATE_DRIVER_SDI: track 16.8 -> 15.1 mm
- net Net-(U8-CPH): track 2.26 -> 4.01 mm
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- added copper zone on F.Cu, net +12V
- added copper zone on In3.Cu, net +12V
- added copper zone on In3.Cu, net +3V3
- added copper zone on F.Cu, net /Motor/Gate Driver/H_BRIDGE_SHA
- added copper zone on F.Cu, net /Motor/Gate Driver/H_BRIDGE_SHB
- added copper zone on F.Cu, net /Motor/Gate Driver/H_BRIDGE_SHC
- added copper zone on In3.Cu, net VBUS
Other:
- outline, holes or cut-outs redrawn

Commit message: fix
Parts:
- added C37: 10u, Capacitor_SMD:C_1210_3225Metric, F.Cu at (105.7, 70.0)
- added C38: 10u, Capacitor_SMD:C_1210_3225Metric, B.Cu at (116.6, 84.1)
- added C39: 10u, Capacitor_SMD:C_1210_3225Metric, F.Cu at (102.2, 77.8)
- added C40: 10u, Capacitor_SMD:C_1210_3225Metric, F.Cu at (116.6, 87.3)
- added C40: 10u, Capacitor_SMD:C_1210_3225Metric, F.Cu at (104.7, 87.3)
- added C41: 10u, Capacitor_SMD:C_1210_3225Metric, B.Cu at (117.0, 79.7)
- added C52: 10u, Capacitor_SMD:C_1210_3225Metric, B.Cu at (136.2, 79.7)
- moved C20 59.7 mm to (123.4, 79.7), turned to 90 degrees
- moved C31 59.6 mm to (126.6, 79.7), turned to 90 degrees
- moved C32 59.6 mm to (129.8, 79.7), turned to 90 degrees
- moved C33 32.7 mm to (116.6, 87.3)
- moved C14 15.6 mm to (120.2, 79.7), turned to 90 degrees
- moved C17 13.0 mm to (133.0, 79.7), turned to 90 degrees
- moved R30 5.79 mm to (120.5, 83.9)
- moved CN3 4.96 mm to (147.3, 71.0)
- moved U17 4.75 mm to (124.2, 85.6)
- moved U9 4.59 mm to (126.2, 71.0)
- moved U16 4.51 mm to (128.5, 85.6)
- moved U14 2.51 mm to (133.1, 85.5)
- moved U15 2.41 mm to (137.6, 85.5)
- moved R29 2.29 mm to (141.2, 85.4)
- moved R28 2.20 mm to (145.3, 85.4)
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Connections:
- CN3 pad 1: /Motor/Gate Driver/H_BRIDGE_SHA -> /Motor/Gate Driver/H_BRIDGE_SHC
- CN3 pad 3: /Motor/Gate Driver/H_BRIDGE_SHC -> /Motor/Gate Driver/H_BRIDGE_SHA
Routing:
- net GND: track 60.5 -> 166.7 mm, vias 186 -> 300
- net /Motor/Gate Driver/H_BRIDGE_SHC: track 19.5 -> 16.1 mm
- net /Motor/Gate Driver/H_BRIDGE_GLC: track 21.1 -> 17.8 mm
- net /Motor/Gate Driver/H_BRIDGE_GHC: track 17.0 -> 14.3 mm
- net /Motor/Gate Driver/H_BRIDGE_GHA: track 12.6 -> 15.1 mm
- net /Motor/Gate Driver/H_BRIDGE_GLB: track 6.86 -> 9.37 mm
- net /Motor/Gate Driver/H_BRIDGE_SPB: track 6.10 -> 8.43 mm
- net VBUS: track 13.4 -> 15.7 mm, vias 157 -> 359
- net /Motor/Gate Driver/H_BRIDGE_GLA: track 8.66 -> 10.8 mm
- net /Motor/Gate Driver/H_BRIDGE_SHA: track 9.52 -> 11.7 mm
- net /Motor/Gate Driver/H_BRIDGE_SPA: track 7.57 -> 9.66 mm
- net /Motor/Gate Driver/H_BRIDGE_SHB: track 4.92 -> 6.96 mm
- net /Motor/Gate Driver/H_BRIDGE_SPC: track 23.6 -> 22.1 mm
- net /Motor/Gate Driver/H_BRIDGE_GHB: track 8.89 -> 10.2 mm
- net +3V3: track 19.3 -> 20.4 mm, vias 17 -> 19
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- added copper zone on B.Cu, net +3V3
- added copper zone on F.Cu, net /Motor/Gate Driver/H_BRIDGE_SPA
- added copper zone on F.Cu, net /Motor/Gate Driver/H_BRIDGE_SPB
- added copper zone on F.Cu, net /Motor/Gate Driver/H_BRIDGE_SPC
Other:
- board size 50 x 47 mm -> 50 x 50 mm

Commit message: fix
Parts:
- C20, C31, C32: moved to F.Cu
- C37, C39: moved to B.Cu
- moved C37 46.6 mm to (150.5, 83.1), turned to 180 degrees
- moved C39 43.7 mm to (145.8, 76.7)
- moved C52 14.2 mm to (150.5, 79.9), turned to 180 degrees
- moved C32 13.4 mm to (116.6, 77.7), turned to 180 degrees
- moved C17 12.8 mm to (145.8, 79.9), turned to 180 degrees
- moved C31 10.1 mm to (116.6, 80.9), turned to 180 degrees
- moved C20 8.11 mm to (116.6, 84.1), turned to 180 degrees
- moved C14 4.12 mm to (116.6, 77.7), turned to 180 degrees
- moved C41 1.28 mm to (116.6, 80.9), turned to 180 degrees
Routing:
- net GND: vias 300 -> 284
- added copper zone on B.Cu, net GND
- added copper zone on B.Cu, net VBUS
