File: electronics/main_board/main_board.kicad_pcb (KiCad board)
At the start: 6 copper layers, 50 x 50 mm, 108 parts, among them CN1 DB141R-2.54-2P, CN3 KF202-5.0-3P, U1 HUSB238A-BB001-QN16R, U10 TJA1051TK/3, U11 NTTFS5C454NL, U13 NTTFS5C454NL, U14 NTTFS5C454NL, U15 NTTFS5C454NL, U16 NTTFS5C454NL, U17 NTTFS5C454NL, U18 TJA1051TK/3, U2 LMR51420YDD, U3 TPS62933DRL, U6 ESP32-S3-WROOM-1, U7 STM32G474VEH6, U8 DRV8323SRTA, U9 AFD01-S35FCA-00

Commit message: fix
Parts:
- removed the C40 at (104.7, 87.3)
- removed U9: AFD01-S35FCA-00, main_board:AFD01-S35FCA-00
- added U22: AFD01-S35FCA-00, main_board:AFD01-S35FCA-00, F.Cu at (126.2, 74.8)
- C21: moved to F.Cu
- moved C17 37.4 mm to (182.9, 75.0)
- moved C39 37.4 mm to (182.9, 71.8)
- moved C37 37.4 mm to (187.6, 78.2)
- moved C52 37.4 mm to (187.6, 75.0)
- moved CN3 4.60 mm to (148.3, 75.5)
- moved REF** 3.50 mm to (161.0, 72.5)
- moved C21 3.05 mm to (145.4, 96.2), turned to 0 degrees
- moved R21 1.07 mm to (128.8, 99.8)
- moved C14 0.91 mm to (116.6, 78.6)
- moved C15 0.91 mm to (116.6, 97.8)
- moved C16 0.91 mm to (116.6, 91.4)
- moved C18 0.91 mm to (116.6, 94.6)
- moved C19 0.91 mm to (116.6, 97.8)
- moved C20 0.91 mm to (116.6, 85.0)
- moved C23 0.91 mm to (116.6, 91.4)
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Connections:
- net /Expansion Port/EXPANSION_IO16 renamed /MCU/EXPANSION_IO16
- net /Expansion Port/EXPANSION_IO8 renamed /MCU/EXPANSION_IO8
- USB1 pad A4B9: Net-(USB1-VBUS) -> /Power/VBUS_IN
- USB1 pad B4A9: Net-(USB1-VBUS) -> /Power/VBUS_IN
Routing:
- net /Expansion Port/EXPANSION_IO45: track 0.00 -> 55.7 mm, vias 0 -> 2
- net /MCU/STM32_EN: track 0.76 -> 53.3 mm
- net /Expansion Port/EXPANSION_IO3: track 0.00 -> 51.4 mm, vias 0 -> 2
- net /Expansion Port/EXPANSION_IO46: track 0.00 -> 49.2 mm, vias 0 -> 2
- net /Expansion Port/EXPANSION_IO9: track 0.00 -> 48.6 mm, vias 0 -> 2
- net /Expansion Port/EXPANSION_IO10: track 0.00 -> 46.0 mm, vias 0 -> 2
- net /Expansion Port/EXPANSION_IO11: track 0.00 -> 45.6 mm, vias 0 -> 2
- net /Expansion Port/EXPANSION_IO12: track 0.00 -> 43.0 mm, vias 0 -> 2
- net /Expansion Port/EXPANSION_IO42: track 0.00 -> 40.0 mm, vias 0 -> 2
- net /Expansion Port/EXPANSION_IO1: track 0.00 -> 39.9 mm, vias 0 -> 2
- net /Expansion Port/EXPANSION_IO41: track 0.00 -> 38.8 mm, vias 0 -> 2
- net /Expansion Port/EXPANSION_IO2: track 0.00 -> 38.6 mm, vias 0 -> 2
- net /Expansion Port/EXPANSION_IO35: track 0.00 -> 36.7 mm, vias 0 -> 2
- net /Expansion Port/EXPANSION_IO37: track 0.00 -> 35.5 mm, vias 0 -> 2
- net /Expansion Port/EXPANSION_IO40: track 0.00 -> 35.4 mm, vias 0 -> 2
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- added copper zone on In4.Cu, net VBUS
- removed copper zone on B.Cu, net +3V3
Other:
- board size 50 x 50 mm -> 50 x 45.5 mm

Commit message: fix
Routing:
- net /Expansion Port/EXPANSION_IO13: track 1.41 -> 60.4 mm, vias 1 -> 2
- net /Expansion Port/EXPANSION_IO14: track 0.86 -> 58.1 mm, vias 1 -> 2
- net /Expansion Port/EXPANSION_IO21: track 1.41 -> 58.5 mm, vias 1 -> 2
- net /Expansion Port/EXPANSION_IO47: track 0.97 -> 56.7 mm, vias 1 -> 2
- net /Expansion Port/EXPANSION_IO48: track 1.42 -> 56.9 mm, vias 1 -> 2
- net /MCU/USB_D+: track 19.3 -> 52.1 mm
- net /MCU/USB_D-: track 23.1 -> 52.4 mm
- net /Expansion Port/ENCODER_SCL: track 0.87 -> 25.8 mm, vias 1 -> 2
- net /Expansion Port/ENCODER_SDA: track 1.43 -> 25.8 mm, vias 1 -> 2
- net Net-(U6-IO0): track 14.2 -> 36.2 mm, vias 0 -> 2
- net GND: track 193.5 -> 174.2 mm, vias 322 -> 404
- net /Expansion Port/EXPANSION_IO12: track 43.0 -> 48.6 mm
- net /Expansion Port/EXPANSION_IO11: track 45.6 -> 50.1 mm
- net /Expansion Port/EXPANSION_IO10: track 46.0 -> 49.8 mm
- net /Expansion Port/EXPANSION_IO9: track 48.6 -> 51.5 mm
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
Commit message: fix
Parts:
- added REF**: , TestPoint:TestPoint_Pad_D1.0mm, F.Cu at (133.3, 123.0)
- added REF**: GND, TestPoint:TestPoint_Pad_D1.0mm, F.Cu at (129.6, 122.8)
- added REF**: , TestPoint:TestPoint_Pad_D1.0mm, F.Cu at (121.4, 122.6)
- added REF**: , TestPoint:TestPoint_Pad_D1.0mm, F.Cu at (125.4, 122.8)
- added REF**: , TestPoint:TestPoint_Pad_D1.0mm, F.Cu at (113.6, 122.7)
Routing:
- net GND: track 174.2 -> 92.0 mm, vias 404 -> 427

Commit message: fix
Parts:
- removed C52: 10u, Capacitor_SMD:C_1210_3225Metric
- removed the REF** at (133.3, 123.0)
- removed the REF** at (129.6, 122.8)
- removed the REF** at (121.4, 122.6)
- removed the REF** at (125.4, 122.8)
- removed the REF** at (113.6, 122.7)
- added REF**: TestPoint_THTPad_D1.0mm_Drill0.5mm, TestPoint:TestPoint_THTPad_D1.0mm_Drill0.5mm, F.Cu at (118.5, 121.5)
- C32: moved to B.Cu
- moved C17 59.3 mm to (123.7, 79.3), turned to 90 degrees
- moved C37 57.4 mm to (130.1, 79.3), turned to 90 degrees
- moved C39 56.5 mm to (126.9, 79.3), turned to 90 degrees
- moved U20 32.3 mm to (109.1, 83.5)
- moved U12 32.3 mm to (109.1, 79.6)
- moved U19 32.3 mm to (109.1, 81.5)
- moved U21 32.3 mm to (109.1, 85.5)
- moved REF** 21.2 mm to (116.3, 77.8)
- moved C32 19.9 mm to (136.6, 79.3), turned to 90 degrees
- moved C14 16.7 mm to (133.3, 79.3), turned to 90 degrees
- moved U22 1.18 mm to (127.4, 74.7)
- moved CN1 0.81 mm to (158.3, 83.3)
Connections:
- REF** pad 1: (no net) -> GND (x4)
Routing:
- net /Expansion Port/EXPANSION_IO45: track 55.1 -> 35.2 mm
- net +3V3: track 45.2 -> 49.2 mm, vias 80 -> 83
- net GND: track 92.0 -> 88.1 mm, vias 427 -> 414
- net /MCU/STM32_EN: track 53.3 -> 51.0 mm, vias 1 -> 3
- net /Expansion Port/EXPANSION_IO35: track 36.1 -> 34.2 mm
- net /Expansion Port/EXPANSION_IO36: track 34.4 -> 32.5 mm
- net /Expansion Port/EXPANSION_IO37: track 34.6 -> 33.0 mm
- net /Expansion Port/EXPANSION_IO21: track 58.5 -> 57.2 mm
- net /Expansion Port/EXPANSION_IO3: track 53.1 -> 51.9 mm
- net /Expansion Port/EXPANSION_IO38: track 33.5 -> 32.2 mm
- net /Expansion Port/EXPANSION_IO46: track 51.5 -> 50.2 mm
- net /Expansion Port/EXPANSION_IO42: track 40.0 -> 38.8 mm
- net /Expansion Port/EXPANSION_IO12: track 48.6 -> 47.4 mm
- net /Expansion Port/EXPANSION_IO47: track 56.7 -> 55.5 mm
- net /Expansion Port/EXPANSION_IO10: track 49.8 -> 48.6 mm
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- added copper zone on In2.Cu, net GND
Other:
- outline, holes or cut-outs redrawn

Commit message: fix
Parts:
- removed the REF** at (118.5, 121.5)
- CN3: value KF202-5.0-3P -> val
- D4: value BZT52C10 -> D_SOD-123F
- REF**: moved to B.Cu
- U22: value AFD01-S35FCA-00 -> val
- USB1: value GT-USB-7004N -> val
- moved R30 3.01 mm to (122.6, 81.8), turned to -90 degrees
- moved CN1 2.84 mm to (158.3, 80.5)
- moved U5 1.47 mm to (125.2, 106.8)
- moved C54 1.16 mm to (135.1, 105.9)
- moved REF** 1.00 mm to (162.0, 72.5)
- moved REF** 1.00 mm to (162.0, 112.0)
- moved C15 0.97 mm to (117.6, 97.8)
- moved C23 0.97 mm to (117.6, 91.4)
- moved C28 0.97 mm to (117.6, 94.6)
- moved C33 0.97 mm to (117.6, 88.2)
- moved C38 0.97 mm to (117.6, 85.0)
- moved C41 0.97 mm to (117.6, 81.8)
- moved C16 0.96 mm to (117.6, 91.4)
- moved C19 0.96 mm to (117.6, 97.8)
- moved C20 0.96 mm to (117.6, 85.0)
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Connections:
- U8 pad 10: GND -> /Motor/Gate Driver/H_BRIDGE_SNA
- U8 pad 11: GND -> /Motor/Gate Driver/H_BRIDGE_SNB
- U8 pad 20: GND -> /Motor/Gate Driver/H_BRIDGE_SNC
Routing:
- net GND: track 88.1 -> 30.6 mm, vias 414 -> 374
- net /Motor/Gate Driver/H_BRIDGE_SNC: track 0.00 -> 26.1 mm, vias 0 -> 2
- net /Motor/Gate Driver/H_BRIDGE_SNA: track 0.00 -> 8.46 mm, vias 0 -> 1
- net /Motor/Gate Driver/H_BRIDGE_SNB: track 0.00 -> 8.33 mm, vias 0 -> 1
- net +3V3: track 49.2 -> 45.4 mm, vias 83 -> 88
- net /Motor/Gate Driver/MOTOR_C_CURRENT_SENSE: track 3.19 -> 5.57 mm
- net /Power/VBUS_IN: track 14.3 -> 12.8 mm
- net /Motor/Gate Driver/H_BRIDGE_SPC: track 22.1 -> 23.6 mm, vias 2 -> 3
- net /Motor/Gate Driver/GATE_DRIVER_INHA: track 17.5 -> 18.9 mm
- net Net-(U3-SW): track 0.24 -> 1.62 mm
- net /Expansion Port/EXPANSION_IO2: track 38.7 -> 39.9 mm
- net /CAN Transceiver1/CAN_TX: track 9.93 -> 8.69 mm
- net /MCU/STM32_EN: track 51.0 -> 52.0 mm
- net Net-(U8-DVDD): track 4.14 -> 5.09 mm
- net Net-(U3-BST): track 0.23 -> 1.18 mm
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Other:
- board size 50 x 45.5 mm -> 51 x 45.5 mm
- rule pad_to_mask_clearance: 0.038 -> 0
- rule solder_mask_min_width: 0.1 -> 0.03
- board text added: "+12V"
- board text added: "+12V Buck"
- board text added: "+3V3"
- board text added: "+3V3 Buck"
- board text added: "CAN BUS"
- board text added: "EN"
- board text added: "Expansion Port"
- board text added: "GND|+12V"
- board text added: "Gate Driver"
- board text added: "H-Bridge"
- board text added: "HackerFab spin coater main board rev 1.0"
- board text added: "IO0"
- board text added: "MCU"
- board text added: "Motor"
- board text added: "Pump"
- board text added: "USB-PD"
- board text added: "VBUS"
- board text added: "VBUSIN"
