File: electronics/main_board/main_board.kicad_pcb (KiCad board)
At the start: 6 copper layers, 51 x 45.5 mm, 106 parts, among them CN1 DB141R-2.54-2P, CN3 val, U1 HUSB238A-BB001-QN16R, U10 TJA1051TK/3, U11 NTTFS5C454NL, U13 NTTFS5C454NL, U14 NTTFS5C454NL, U15 NTTFS5C454NL, U16 NTTFS5C454NL, U17 NTTFS5C454NL, U18 TJA1051TK/3, U2 LMR51420YDD, U22 val, U3 TPS62933DRL, U6 ESP32-S3-WROOM-1, U7 STM32G474VEH6, U8 DRV8323SRTA

Commit message: fix
Parts:
- removed U12, U19, U20, U21: ~, main_board:XL-1005UOC
- CN3: value val -> KF202-5.0-3P
- D4: value D_SOD-123F -> BZT52C10
- U22: value val -> AFD01-S35FCA-00
- USB1: value val -> GT-USB-7004N
- moved REF** 1.50 mm to (162.0, 71.0)
Connections:
- U8 pad 10: /Motor/Gate Driver/H_BRIDGE_SNA -> GND
- U8 pad 11: /Motor/Gate Driver/H_BRIDGE_SNB -> GND
- U8 pad 20: /Motor/Gate Driver/H_BRIDGE_SNC -> GND
Routing:
- net GND: track 30.6 -> 73.5 mm, vias 374 -> 378
- net /Motor/Gate Driver/H_BRIDGE_SNC: track 26.1 -> 0.00 mm, vias 2 -> 0
- net /Motor/Gate Driver/H_BRIDGE_SNA: track 8.46 -> 0.00 mm, vias 1 -> 0
- net /Motor/Gate Driver/H_BRIDGE_SNB: track 8.33 -> 0.00 mm, vias 1 -> 0
Other:
- board size 51 x 45.5 mm -> 51 x 47 mm

Commit message: fix
Connections:
- U22 pad 21: /Expansion Port/EXPANSION_IO9 -> /Expansion Port/STM32-SWDIO
- U22 pad 22: /Expansion Port/EXPANSION_IO46 -> /Expansion Port/STM32-SWCLK
- U22 pad 23: /Expansion Port/EXPANSION_IO3 -> /Expansion Port/STM32-BOOT0
- U7 pad A3: unconnected-(U7A-PB8-BOOT0-PadA3) -> /Expansion Port/STM32-BOOT0
- U7 pad C9: unconnected-(U7A-PA12-PadC9) -> /Expansion Port/STM32-SWDIO
- U7 pad D8: unconnected-(U7A-PA13-PadD8) -> /Expansion Port/STM32-SWCLK
Routing:
- net /Expansion Port/EXPANSION_IO3: track 51.6 -> 0.00 mm, vias 2 -> 0
- net /Expansion Port/EXPANSION_IO9: track 50.4 -> 0.00 mm, vias 2 -> 0
- net /Expansion Port/EXPANSION_IO46: track 50.2 -> 0.00 mm, vias 2 -> 0
- net /Expansion Port/STM32-BOOT0: track 0.00 -> 28.0 mm, vias 0 -> 2
- net /Expansion Port/STM32-SWCLK: track 0.00 -> 22.5 mm, vias 0 -> 2
- net /Expansion Port/STM32-SWDIO: track 0.00 -> 22.4 mm, vias 0 -> 2
- net Net-(U6-IO0): track 35.6 -> 36.7 mm
- net GND: track 73.5 -> 72.5 mm
- net /Motor/Gate Driver/H_BRIDGE_SPC: track 23.6 -> 22.7 mm
- net VBUS: vias 356 -> 350
