File: electronics/main_board/H-Bridge.kicad_sch (KiCad schematic)
At the start: 10 parts, among them J1 Screw_Terminal_01x03, U11 NTTFS5C454NL, U13 NTTFS5C454NL, U14 NTTFS5C454NL, U15 NTTFS5C454NL, U16 NTTFS5C454NL, U17 NTTFS5C454NL

Commit message: fix
Connections:
- net H_BRIDGE_SHA: now also U13.10, U13.11, U13.9
- net H_BRIDGE_SHB: now also U15.10, U15.11, U15.9
- net H_BRIDGE_SHC: now also U17.10, U17.11, U17.9
- net VBUS: now also U11.10, U11.11, U11.9, U14.10, U14.11, U14.9, U16.10, U16.11, U16.9
Changed lines of the file:
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@@
+	(wire
+		(pts
+			(xy 93.98 50.8) (xy 93.98 53.34)
+		)
+		(stroke
+			(width 0)
+			(type default)
+		)
+	)
 	(wire
 		(pts
@@
 		(pts
 			(xy 154.94 50.8) (xy 215.9 50.8)
-		)
-		(stroke
-			(width 0)
-			(type default)
-		)
-	)
-	(wire
-		(pts
-			(xy 93.98 50.8) (xy 93.98 53.34)
 		)
 		(stroke
@@
 		(pin "6"
 		)
+		(pin "10"
+		)
+		(pin "11"
+		)
+		(pin "9"
+		)
 		(instances
 			(project "main_board"
@@
 		(pin "6"
 		)
+		(pin "10"
+		)
+		(pin "9"
+		)
+		(pin "11"
+		)
 		(instances
-			(project ""
+			(project "main_board"
 				(path "/82f7d8d0-a6dd-48aa-80fa-49fc2cccb16f/c9ec9ccd-2e72-4236-908b-58c2b4d5f776/effaf589-d03b-428f-9cd2-be6913714a7d"
 					(reference "U11")
@@
 		(pin "6"
 		)
+		(pin "10"
+		)
+		(pin "11"
+		)
+		(pin "9"
+		)
 		(instances
 			(project "main_board"
@@
 		(pin "6"
 		)
+		(pin "10"
+		)
+		(pin "11"
+		)
+		(pin "9"
+		)
 		(instances
 			(project "main_board"
@@
 		(pin "6"
 		)
+		(pin "10"
+		)
+		(pin "11"
+		)
+		(pin "9"
+		)
 		(instances
 			(project "main_board"
@@
 		)
 		(instances
-			(project ""
+			(project "main_board"
 				(path "/82f7d8d0-a6dd-48aa-80fa-49fc2cccb16f/c9ec9ccd-2e72-4236-908b-58c2b4d5f776/effaf589-d03b-428f-9cd2-be6913714a7d"
 					(reference "J1")
@@
 		(pin "6"
 		)
+		(pin "10"
+		)
+		(pin "11"
+		)
+		(pin "9"
+		)
 		(instances
 			(project "main_board"
@@
 		)
 		(instances
-			(project ""
+			(project "main_board"
 				(path "/82f7d8d0-a6dd-48aa-80fa-49fc2cccb16f/c9ec9ccd-2e72-4236-908b-58c2b4d5f776/effaf589-d03b-428f-9cd2-be6913714a7d"
 					(reference "#PWR016")

Commit message: fix
Parts:
- removed J1: Screw_Terminal_01x03, symbol Connector:Screw_Terminal_01x03
Changed lines of the file:
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@@
 	(wire
 		(pts
-			(xy 93.98 66.04) (xy 106.68 66.04)
+			(xy 93.98 66.04) (xy 111.76 66.04)
 		)
 		(stroke
@@
 	(wire
 		(pts
-			(xy 215.9 66.04) (xy 228.6 66.04)
+			(xy 215.9 66.04) (xy 233.68 66.04)
 		)
 		(stroke
@@
 	(wire
 		(pts
-			(xy 149.86 127) (xy 137.16 127)
-		)
-		(stroke
-			(width 0)
-			(type default)
-		)
-	)
-	(wire
-		(pts
 			(xy 88.9 58.42) (xy 86.36 58.42)
 		)
@@
 	(wire
 		(pts
-			(xy 149.86 129.54) (xy 137.16 129.54)
-		)
-		(stroke
-			(width 0)
-			(type default)
-		)
-	)
-	(wire
-		(pts
 			(xy 147.32 91.44) (xy 154.94 91.44)
 		)
@@
 	(wire
 		(pts
-			(xy 149.86 132.08) (xy 137.16 132.08)
-		)
-		(stroke
-			(width 0)
-			(type default)
-		)
-	)
-	(wire
-		(pts
 			(xy 215.9 48.26) (xy 215.9 50.8)
 		)
@@
 	(wire
 		(pts
+			(xy 154.94 66.04) (xy 172.72 66.04)
+		)
+		(stroke
+			(width 0)
+			(type default)
+		)
+	)
+	(wire
+		(pts
 			(xy 215.9 78.74) (xy 215.9 81.28)
 		)
@@
 	(wire
 		(pts
-			(xy 154.94 66.04) (xy 167.64 66.04)
-		)
-		(stroke
-			(width 0)
-			(type default)
-		)
-	)
-	(wire
-		(pts
 			(xy 208.28 66.04) (xy 215.9 66.04)
 		)
@@
 			(width 0)
 			(type default)
-		)
-	)
-	(label "MOTOR_A"
-		(at 106.68 66.04 180)
-		(effects
-			(font
-				(size 1.27 1.27)
-			)
-			(justify right bottom)
-		)
-	)
-	(label "MOTOR_C"
-		(at 228.6 66.04 180)
-		(effects
-			(font
-				(size 1.27 1.27)
-			)
-			(justify right bottom)
-		)
-	)
-	(label "MOTOR_C"
-		(at 137.16 132.08 0)
-		(effects
-			(font
-				(size 1.27 1.27)
-			)
-			(justify left bottom)
-		)
-	)
-	(label "MOTOR_B"
-		(at 167.64 66.04 180)
-		(effects
-			(font
-				(size 1.27 1.27)
-			)
-			(justify right bottom)
-		)
-	)
-	(label "MOTOR_A"
-		(at 137.16 127 0)
-		(effects
-			(font
-				(size 1.27 1.27)
-			)
-			(justify left bottom)
-		)
-	)
-	(label "MOTOR_B"
-		(at 137.16 129.54 0)
-		(effects
-			(font
-				(size 1.27 1.27)
-			)
-			(justify left bottom)
 		)
 	)
@@
 		)
 	)
+	(hierarchical_label "MOTOR_C"
+		(shape bidirectional)
+		(at 233.68 66.04 0)
+		(effects
+			(font
+				(size 1.27 1.27)
+			)
+			(justify left)
+		)
+	)
 	(hierarchical_label "H_BRIDGE_SHA"
 		(shape output)
@@
 		)
 	)
+	(hierarchical_label "MOTOR_B"
+		(shape bidirectional)
+		(at 172.72 66.04 0)
+		(effects
+			(font
+				(size 1.27 1.27)
+			)
+			(justify left)
+		)
+	)
 	(hierarchical_label "H_BRIDGE_SNC"
 		(shape output)
@@
 			)
 			(justify right)
+		)
+	)
+	(hierarchical_label "MOTOR_A"
+		(shape bidirectional)
+		(at 111.76 66.04 0)
+		(effects
+			(font
+				(size 1.27 1.27)
+			)
+			(justify left)
 		)
 	)
@@
 					(unit 1)
 				)
-			)
-		)
-	)
-	(symbol
-		(lib_id "Connector:Screw_Terminal_01x03")
-		(at 154.94 129.54 0)
-		(unit 1)
-		(exclude_from_sim no)
-		(in_bom yes)
-		(on_board yes)
-		(dnp no)
-		(fields_autoplaced yes)
-		(property "Reference" "J1"
-			(at 157.48 128.2699 0)
-			(effects
-				(font
-					(size 1.27 1.27)
-				)
-				(justify left)
-			)
-		)
-		(property "Value" "Screw_Terminal_01x03"
-			(at 157.48 130.8099 0)
-			(effects
-				(font
-					(size 1.27 1.27)
-				)
-				(justify left)
-			)
-		)
-		(property "Footprint" ""
-			(at 154.94 129.54 0)
-			(effects
-				(font
-					(size 1.27 1.27)
-				)
-				(hide yes)
-			)
-		)
-		(property "Datasheet" "~"
-			(at 154.94 129.54 0)
-			(effects
-				(font
-					(size 1.27 1.27)
-				)
-				(hide yes)
-			)
-		)
-		(property "Description" "Generic screw terminal, single row, 01x03, script generated (kicad-library-utils/schlib/autogen/connector/)"
-			(at 154.94 129.54 0)
-			(effects
-				(font
-					(size 1.27 1.27)
-				)
-				(hide yes)
-			)
-		)
-		(pin "3"
-		)
-		(pin "2"
-		)
-		(pin "1"
-		)
-		(instances
-			(project "main_board"
-				(path "/82f7d8d0-a6dd-48aa-80fa-49fc2cccb16f/c9ec9ccd-2e72-4236-908b-58c2b4d5f776/effaf589-d03b-428f-9cd2-be6913714a7d"
-					(reference "J1")
-					(unit 1)
-				)

Commit message: fix
Parts:
- added NT1, NT2, NT3: NetTie_2, NetTie:NetTie-2_SMD_Pad0.5mm, symbol Device:NetTie_2
Connections:
- net GND: now also NT1.2, NT2.2, NT3.2
- new net H_BRIDGE_SNA: NT1.1
- new net H_BRIDGE_SNB: NT2.1
- new net H_BRIDGE_SNC: NT3.1

Commit message: fix
Parts:
- removed NT1, NT2, NT3: NetTie_2, NetTie:NetTie-2_SMD_Pad0.5mm, symbol Device:NetTie_2
