File: electronics/main_board/MCU.kicad_sch (KiCad schematic)
At the start: 8 parts, among them U6 ESP32-S3-WROOM-1

Commit message: fix
Connections:
- net CAN_RX: now also U6.7 (IO7); no longer U6.26 (IO45)
- net CAN_TX: now also U6.8 (IO15); no longer U6.35 (IO42)
- net EN_12V: now also U6.4 (IO4); no longer U6.8 (IO15)
- net PD_FAULT: now also U6.6 (IO6); no longer U6.16 (IO46)
- net PD_INT_N: now also U6.5 (IO5); no longer U6.15 (IO3)
- net EXPANSION_IO8: now reaches U6.12 (IO8)
- net EXPANSION_IO9: now reaches U6.17 (IO9)
- net EXPANSION_IO10: now reaches U6.18 (IO10)
- net EXPANSION_IO11: now reaches U6.19 (IO11)
- net EXPANSION_IO12: now reaches U6.20 (IO12)
- net EXPANSION_IO13: now reaches U6.21 (IO13)
- net EXPANSION_IO14: now reaches U6.22 (IO14)
- net EXPANSION_IO21: now reaches U6.23 (IO21)
- net EXPANSION_IO47: now reaches U6.24 (IO47)
- net EXPANSION_IO48: now reaches U6.25 (IO48)
- net EXPANSION_IO35: now reaches U6.28 (IO35)
- net EXPANSION_IO36: now reaches U6.29 (IO36)
- net EXPANSION_IO37: now reaches U6.30 (IO37)
- net EXPANSION_IO38: now reaches U6.31 (IO38)
- net EXPANSION_IO40: now reaches U6.33 (IO40)
- net EXPANSION_IO41: now reaches U6.34 (IO41)
- net EXPANSION_IO2: now reaches U6.38 (IO2)
- net EXPANSION_IO1: now reaches U6.39 (IO1)
- net EXPANSION_IO16: now reaches U6.9 (IO16)
- new net EXPANSION_IO3: U6.15 (IO3)
- new net EXPANSION_IO42: U6.35 (IO42)
- new net EXPANSION_IO45: U6.26 (IO45)
- new net EXPANSION_IO46: U6.16 (IO46)

Commit message: fix
Parts:
- added R40, R41, R42, R43: 10k, Resistor_SMD:R_0402_1005Metric, symbol Device:R
Connections:
- net +3V3: now also R40.1, R41.1, R42.1, R43.1
- net PD_SCL: now also R41.2, R43.2
- net PD_SDA: now also R40.2, R42.2
