File: electronics/main_board/Motor Connector.kicad_sch (KiCad schematic)
At the start: 1 part, among them CN3 KF202-5.0-3P

Commit message: fix
Connections:
- net MOTOR_A: now also CN3.3; no longer CN3.1
- net MOTOR_C: now also CN3.1; no longer CN3.3
Changed lines of the file:
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@@
-	(wire
-		(pts
-			(xy 127 78.74) (xy 132.08 78.74)
-		)
-		(stroke
-			(width 0)
-			(type default)
-		)
-	)
 	(wire
 		(pts
@@
 		)
 	)
+	(wire
+		(pts
+			(xy 127 78.74) (xy 132.08 78.74)
+		)
+		(stroke
+			(width 0)
+			(type default)
+		)
+	)
+	(hierarchical_label "MOTOR_C"
+		(shape bidirectional)
+		(at 127 78.74 180)
+		(effects
+			(font
+				(size 1.27 1.27)
+			)
+			(justify right)
+		)
+	)
 	(hierarchical_label "MOTOR_B"
 		(shape bidirectional)
@@
 		)
 	)
-	(hierarchical_label "MOTOR_C"
+	(hierarchical_label "MOTOR_A"
 		(shape bidirectional)
 		(at 127 83.82 180)
 		(effects
 			(font
-				(size 1.27 1.27)
-			)
-			(justify right)
-		)
-	)
-	(hierarchical_label "MOTOR_A"
-		(shape bidirectional)
-		(at 127 78.74 180)
-		(effects
-			(font
