File: electronics/main_board/STM32.kicad_sch (KiCad schematic)
At the start: 9 parts, among them U7 STM32G474VEH6

Commit message: fix
Connections:
- net STM32-BOOT0: now reaches U7.A3 (PB8-BOOT0)
- net STM32-SWDIO: now reaches U7.C9 (PA12)
- net STM32-SWCLK: now reaches U7.D8 (PA13)
Changed lines of the file:
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@@
+	(wire
+		(pts
+			(xy 119.38 63.5) (xy 116.84 63.5)
+		)
+		(stroke
+			(width 0)
+			(type default)
+		)
+	)
 	(wire
 		(pts
@@
 	(wire
 		(pts
+			(xy 119.38 96.52) (xy 116.84 96.52)
+		)
+		(stroke
+			(width 0)
+			(type default)
+		)
+	)
+	(wire
+		(pts
 			(xy 109.22 162.56) (xy 111.76 162.56)
 		)
@@
 	(wire
 		(pts
+			(xy 119.38 66.04) (xy 116.84 66.04)
+		)
+		(stroke
+			(width 0)
+			(type default)
+		)
+	)
+	(wire
+		(pts
 			(xy 160.02 68.58) (xy 165.1 68.58)
 		)
@@
 		(shape output)
 		(at 116.84 60.96 180)
+		(effects
+			(font
+				(size 1.27 1.27)
+			)
+			(justify right)
+		)
+	)
+	(hierarchical_label "STM32-BOOT0"
+		(shape output)
+		(at 116.84 96.52 180)
+		(effects
+			(font
+				(size 1.27 1.27)
+			)
+			(justify right)
+		)
+	)
+	(hierarchical_label "STM32-SWCLK"
+		(shape output)
+		(at 116.84 66.04 180)
 		(effects
 			(font
@@
 		)
 	)
+	(hierarchical_label "STM32-SWDIO"
+		(shape bidirectional)
+		(at 116.84 63.5 180)
+		(effects
+			(font
+				(size 1.27 1.27)
+			)
+			(justify right)
+		)
+	)
