File: electronics/main_board/main_board.kicad_sch (KiCad schematic)
At the start: 1 part, among them J2 Conn_01x30_Socket

Commit message: fix
Parts:
- removed J2: Conn_01x30_Socket, symbol Connector:Conn_01x30_Socket
Other:
- sheet motor renamed Motor
- added sheet Expansion Port (Expansion Port.kicad_sch)
- sheet MCU ports: added EXPANSION_IO1, EXPANSION_IO10, EXPANSION_IO11, EXPANSION_IO12, EXPANSION_IO13, EXPANSION_IO14, EXPANSION_IO16, EXPANSION_IO2, EXPANSION_IO21, EXPANSION_IO3, EXPANSION_IO35, EXPANSION_IO36, EXPANSION_IO37, EXPANSION_IO38, EXPANSION_IO40, EXPANSION_IO41, EXPANSION_IO42, EXPANSION_IO45, EXPANSION_IO46, EXPANSION_IO47, EXPANSION_IO48, EXPANSION_IO8, EXPANSION_IO9; removed none
- sheet Motor: file motor.kicad_sch -> Motor.kicad_sch
- sheet Motor ports: added ENCODER_SCL, ENCODER_SDA; removed none
- sheet Power: file power.kicad_sch -> Power.kicad_sch

Commit message: fix
Other:
- added sheet Pump (Pump.kicad_sch)
Changed lines of the file:
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@@
+	)
+	(sheet
+		(at 210.82 27.94)
+		(size 40.64 25.4)
+		(exclude_from_sim no)
+		(in_bom yes)
+		(on_board yes)
+		(dnp no)
+		(fields_autoplaced yes)
+		(stroke
+			(width 0.1524)
+			(type solid)
+		)
+		(fill
+			(color 0 0 0 0.0000)
+		)
+		(property "Sheetname" "Pump"
+			(at 210.82 27.2284 0)
+			(effects
+				(font
+					(size 1.27 1.27)
+				)
+				(justify left bottom)
+			)
+		)
+		(property "Sheetfile" "Pump.kicad_sch"
+			(at 210.82 53.9246 0)
+			(effects
+				(font
+					(size 1.27 1.27)
+				)
+				(justify left top)
+			)
+		)
+		(instances
+			(project "main_board"
+				(path "/82f7d8d0-a6dd-48aa-80fa-49fc2cccb16f"
+					(page "14")
+				)
+			)
+		)
 	)
 	(sheet

Commit message: fix
Changed lines of the file:
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@@
 		)
 	)
-	(label "CANL"
+	(label "CAN_N"
 		(at 152.4 78.74 0)
 		(effects
@@
 		)
 	)
-	(label "CANH"
+	(label "CAN_P"
 		(at 152.4 76.2 0)
 		(effects

Commit message: fix
Other:
- sheet Expansion Port ports: added STM32-BOOT0, STM32-SWCLK, STM32-SWDIO; removed none
- sheet Motor ports: added STM32-BOOT0, STM32-SWCLK, STM32-SWDIO; removed none
Changed lines of the file:
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@@
+	(wire
+		(pts
+			(xy 233.68 76.2) (xy 248.92 76.2)
+		)
+		(stroke
+			(width 0)
+			(type default)
+		)
+	)
+	(wire
+		(pts
+			(xy 233.68 78.74) (xy 248.92 78.74)
+		)
+		(stroke
+			(width 0)
+			(type default)
+		)
+	)
 	(wire
 		(pts
@@
 	(wire
 		(pts
-			(xy 233.68 71.12) (xy 248.92 71.12)
+			(xy 233.68 66.04) (xy 248.92 66.04)
 		)
 		(stroke
@@
 	(wire
 		(pts
+			(xy 233.68 68.58) (xy 248.92 68.58)
+		)
+		(stroke
+			(width 0)
+			(type default)
+		)
+	)
+	(wire
+		(pts
+			(xy 109.22 114.3) (xy 248.92 114.3)
+		)
+		(stroke
+			(width 0)
+			(type default)
+		)
+	)
+	(wire
+		(pts
+			(xy 109.22 99.06) (xy 248.92 99.06)
+		)
+		(stroke
+			(width 0)
+			(type default)
+		)
+	)
+	(wire
+		(pts
+			(xy 43.18 58.42) (xy 78.74 58.42)
+		)
+		(stroke
+			(width 0)
+			(type default)
+		)
+	)
+	(wire
+		(pts
+			(xy 152.4 48.26) (xy 160.02 48.26)
+		)
+		(stroke
+			(width 0)
+			(type default)
+		)
+	)
+	(wire
+		(pts
 			(xy 233.68 73.66) (xy 248.92 73.66)
-		)
-		(stroke
-			(width 0)
-			(type default)
-		)
-	)
-	(wire
-		(pts
-			(xy 109.22 114.3) (xy 248.92 114.3)
-		)
-		(stroke
-			(width 0)
-			(type default)
-		)
-	)
-	(wire
-		(pts
-			(xy 109.22 99.06) (xy 248.92 99.06)
-		)
-		(stroke
-			(width 0)
-			(type default)
-		)
-	)
-	(wire
-		(pts
-			(xy 43.18 58.42) (xy 78.74 58.42)
-		)
-		(stroke
-			(width 0)
-			(type default)
-		)
-	)
-	(wire
-		(pts
-			(xy 152.4 48.26) (xy 160.02 48.26)
 		)
 		(stroke
@@
 	)
 	(sheet
-		(at 248.92 66.04)
-		(size 25.4 83.82)
+		(at 248.92 58.42)
+		(size 25.4 91.44)
 		(exclude_from_sim no)
 		(in_bom yes)
@@
 		)
 		(property "Sheetname" "Expansion Port"
-			(at 248.92 65.3284 0)
+			(at 248.92 57.7084 0)
 			(effects
 				(font
@@
 		)
 		(pin "ENCODER_SCL" input
-			(at 248.92 71.12 180)
+			(at 248.92 66.04 180)
 			(effects
 				(font
@@
 		)
 		(pin "ENCODER_SDA" bidirectional
-			(at 248.92 73.66 180)
+			(at 248.92 68.58 180)
 			(effects
 				(font
@@
 		(pin "EXPANSION_IO48" bidirectional
 			(at 248.92 147.32 180)
+			(effects
+				(font
+					(size 1.27 1.27)
+				)
+				(justify left)
+			)
+		)
+		(pin "STM32-BOOT0" output
+			(at 248.92 73.66 180)
+			(effects
+				(font
+					(size 1.27 1.27)
+				)
+				(justify left)
+			)
+		)
+		(pin "STM32-SWCLK" output
+			(at 248.92 76.2 180)
+			(effects
+				(font
+					(size 1.27 1.27)
+				)
+				(justify left)
+			)
+		)
+		(pin "STM32-SWDIO" bidirectional
+			(at 248.92 78.74 180)
 			(effects
 				(font
@@
 	)
 	(sheet
-		(at 200.66 66.04)
-		(size 33.02 15.24)
+		(at 200.66 63.5)
+		(size 33.02 17.78)
 		(exclude_from_sim no)
 		(in_bom yes)
@@
 		)
 		(property "Sheetname" "Motor"
-			(at 200.66 65.3284 0)
+			(at 200.66 62.7884 0)
 			(effects
 				(font
@@
 		)
 		(pin "ENCODER_SCL" output
-			(at 233.68 71.12 0)
+			(at 233.68 66.04 0)
 			(effects
 				(font
@@
 		)
 		(pin "ENCODER_SDA" bidirectional
+			(at 233.68 68.58 0)
+			(effects
+				(font
+					(size 1.27 1.27)
+				)
+				(justify right)
+			)
+		)
+		(pin "STM32-BOOT0" output
 			(at 233.68 73.66 0)
 			(effects
 				(font
+					(size 1.27 1.27)
+				)
+				(justify right)
+			)
+		)
+		(pin "STM32-SWCLK" output
+			(at 233.68 76.2 0)
+			(effects
+				(font
+					(size 1.27 1.27)
+				)
+				(justify right)
+			)
+		)
+		(pin "STM32-SWDIO" bidirectional
+			(at 233.68 78.74 0)
+			(effects
+				(font
