File: electronics/io_board/io_board.kicad_pcb (KiCad board)
At the start: 2 copper layers, 80 x 100 mm, 21 parts, among them SW1 PEC11R-4220F-S0024, SW2 PEC11R-4220F-S0024, SW3 MX1A-11NW, SW4 MX1A-11NW, U1 AFD01-S35FCA-00, U2 HS1602A-B, U3 ZX-PZ1.27-2-5PZZ

Commit message: fix
Parts:
- removed C29: 1u, Capacitor_SMD:C_0402_1005Metric
- added C1: 100n, Capacitor_SMD:C_0402_1005Metric, B.Cu at (156.7, 41.7)
- added REF**: MountingHole_2.2mm_M2_DIN965_Pad, MountingHole:MountingHole_2.2mm_M2_DIN965_Pad, F.Cu at (108.0, 18.0)
- added REF**: MountingHole_2.2mm_M2_DIN965_Pad, MountingHole:MountingHole_2.2mm_M2_DIN965_Pad, F.Cu at (182.0, 112.0)
- added REF**: MountingHole_2.2mm_M2_DIN965_Pad, MountingHole:MountingHole_2.2mm_M2_DIN965_Pad, F.Cu at (182.0, 18.0)
- added REF**: MountingHole_2.2mm_M2_DIN965_Pad, MountingHole:MountingHole_2.2mm_M2_DIN965_Pad, F.Cu at (108.0, 112.0)
- C56, FPC1, U1: moved to B.Cu
- moved R10 157.3 mm to (142.4, 69.3), turned to 90 degrees
- moved R12 154.7 mm to (141.4, 69.3), turned to 90 degrees
- moved R11 154.6 mm to (140.4, 69.3), turned to -90 degrees
- moved U3 153.4 mm to (145.0, 60.6)
- moved FPC1 101.1 mm to (145.1, 30.0), turned to 180 degrees
- moved BUZZER1 92.0 mm to (145.0, 89.2), turned to 180 degrees
- moved C56 83.3 mm to (146.1, 26.4), turned to 180 degrees
- moved R1 79.3 mm to (144.5, 69.3), turned to 90 degrees
- moved U1 78.7 mm to (160.0, 35.9), turned to 90 degrees
- moved R38 77.8 mm to (143.5, 69.3), turned to 90 degrees
- moved R4 47.4 mm to (149.6, 69.3), turned to -90 degrees
- moved R5 46.0 mm to (148.5, 69.3), turned to -90 degrees
- moved R6 44.7 mm to (147.5, 69.3), turned to -90 degrees
- moved R3 44.0 mm to (145.5, 69.3), turned to 90 degrees
- moved R7 43.5 mm to (146.5, 69.3), turned to -90 degrees
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Connections:
- BUZZER1 pad 1: /EXPANSION_IO45 -> /EXPANSION_IO47
- C56 pad 1: unconnected-(C56-Pad1) -> +3V3
- C56 pad 2: unconnected-(C56-Pad2) -> GND
- R1 pad 2: /EXPANSION_IO48 -> /EXPANSION_IO45
- R38 pad 2: /EXPANSION_IO47 -> /EXPANSION_IO48
- SW1 pad 1: /EXPANSION_IO10 -> /EXPANSION_IO14
- SW1 pad 3: /EXPANSION_IO11 -> /EXPANSION_IO21
- SW1 pad 4: /EXPANSION_IO12 -> /EXPANSION_IO13
- SW2 pad 1: /EXPANSION_IO13 -> /EXPANSION_IO36
- SW2 pad 3: /EXPANSION_IO14 -> /EXPANSION_IO37
- SW2 pad 4: /EXPANSION_IO21 -> /EXPANSION_IO35
- SW3 pad 1: /EXPANSION_IO47 -> /EXPANSION_IO48
- SW4 pad 1: /EXPANSION_IO48 -> /EXPANSION_IO45
- U1 pad 21: /STM32-SWDIO -> /STM32_SWDIO
- U1 pad 22: /STM32-SWCLK -> /STM32_SWCLK
- U1 pad 23: /STM32-BOOT0 -> /STM32_BOOT0
- U2 pad 11: /EXPANSION_IO38 -> /EXPANSION_IO40
- U2 pad 12: /EXPANSION_IO37 -> /EXPANSION_IO38
- U2 pad 13: /EXPANSION_IO36 -> /EXPANSION_IO41
- U2 pad 14: /EXPANSION_IO35 -> /EXPANSION_IO42
- U2 pad 4: /EXPANSION_IO41 -> /EXPANSION_IO1
- U2 pad 6: /EXPANSION_IO40 -> /EXPANSION_IO2
- U3 pad 1: unconnected-(U3-Pad1) -> /STM32_BOOT0
- U3 pad 10: unconnected-(U3-Pad10) -> GND
- U3 pad 2: unconnected-(U3-Pad2) -> /STM32_SWCLK
- U3 pad 3: unconnected-(U3-Pad3) -> /EXPANSION_IO12
- U3 pad 4: unconnected-(U3-Pad4) -> /STM32_SWDIO
- U3 pad 5: unconnected-(U3-Pad5) -> /EXPANSION_IO11
- U3 pad 6: unconnected-(U3-Pad6) -> VBUS
- U3 pad 7: unconnected-(U3-Pad7) -> +3V3
- U3 pad 8: unconnected-(U3-Pad8) -> /EXPANSION_IO10
- U3 pad 9: unconnected-(U3-Pad9) -> GND
Routing:
- net /EXPANSION_IO48: track 0.00 -> 171.7 mm, vias 0 -> 2
- net /EXPANSION_IO45: track 0.00 -> 138.9 mm, vias 0 -> 2
- net /EXPANSION_IO37: track 0.00 -> 112.6 mm
- net /EXPANSION_IO36: track 0.00 -> 98.4 mm
- net /EXPANSION_IO47: track 0.00 -> 92.3 mm
- net /EXPANSION_IO35: track 0.00 -> 75.4 mm
- net /EXPANSION_IO12: track 0.00 -> 57.1 mm
- net /EXPANSION_IO21: track 0.00 -> 57.1 mm
- net /STM32_SWDIO: track 0.00 -> 57.0 mm
- net /STM32_SWCLK: track 0.00 -> 56.9 mm
- net /EXPANSION_IO14: track 0.00 -> 56.2 mm
- net /EXPANSION_IO11: track 0.00 -> 52.3 mm
- net /EXPANSION_IO10: track 0.00 -> 46.7 mm
- net /STM32_BOOT0: track 0.00 -> 40.9 mm, vias 0 -> 1
- net /EXPANSION_IO13: track 0.00 -> 39.8 mm
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- added copper zone on B.Cu, net +3V3
- added copper zone on F.Cu, net +3V3
- added copper zone on B.Cu, net GND
- added copper zone on F.Cu, net GND
- added copper zone on B.Cu, net VBUS
- added copper zone on F.Cu, net VBUS
Other:
- board size 80 x 100 mm -> 81 x 100.5 mm
- board text added: "+"
- board text added: "100n"
- board text added: "10k"
- board text added: "120"
- board text added: "BOOTO|SWCLK I012 |SWDIO I011 | VBUS +3V3 | IO10 GND | GND"
- board text added: "HackerFab spin coater io board rev 1.0"
- board text added: "SPINNING - RPM: 4K RPM | DURATION: 30S"

Commit message: fix
Parts:
- C1: moved to F.Cu
- moved C1 5.08 mm to (151.6, 41.7)
- moved U3 4.80 mm to (140.5, 62.3), turned to 90 degrees
Connections:
- REF** pad 1: (no net) -> GND (x3)
- U3 pad 1: /STM32_BOOT0 -> GND
- U3 pad 10: GND -> /STM32_SWDIO
- U3 pad 2: /STM32_SWCLK -> GND
- U3 pad 3: /EXPANSION_IO12 -> /STM32_BOOT0
- U3 pad 4: /STM32_SWDIO -> +3V3
- U3 pad 5: /EXPANSION_IO11 -> /EXPANSION_IO12
- U3 pad 7: +3V3 -> /EXPANSION_IO11
- U3 pad 8: /EXPANSION_IO10 -> /STM32_SWCLK
- U3 pad 9: GND -> /EXPANSION_IO10
Routing:
- net /STM32_SWDIO: track 57.0 -> 53.3 mm
- net /STM32_SWCLK: track 56.9 -> 53.4 mm
- net /EXPANSION_IO10: track 46.7 -> 50.1 mm
- net /STM32_BOOT0: track 40.9 -> 39.3 mm
- net /EXPANSION_IO11: track 52.3 -> 53.4 mm
- net Net-(U2-LED+): track 15.9 -> 16.1 mm, vias 0 -> 2
- net VBUS: vias 10 -> 0
- net GND: vias 182 -> 175
- net +3V3: vias 17 -> 13
- removed copper zone on F.Cu, net VBUS
Other:
- board size 81 x 100.5 mm -> 81.3 x 100.7 mm
- board text added: "SWDIO| IO10 SWCLK| IO11 VBUS | I012 +3V3 |BOOT0 GND | GND"
- board text removed: "BOOTO|SWCLK I012 |SWDIO I011 | VBUS +3V3 | IO10 GND | GND"

Commit message: fix
Parts:
- moved C56 0.41 mm to (146.1, 26.8)
- moved C1 0.28 mm to (151.6, 41.5)
- turned U2 to 0 degrees
Connections:
- U2 pad 11: /EXPANSION_IO40 -> /EXPANSION_IO2
- U2 pad 12: /EXPANSION_IO38 -> /EXPANSION_IO1
- U2 pad 13: /EXPANSION_IO41 -> /EXPANSION_IO38
- U2 pad 14: /EXPANSION_IO42 -> /EXPANSION_IO40
- U2 pad 4: /EXPANSION_IO1 -> /EXPANSION_IO41
- U2 pad 6: /EXPANSION_IO2 -> /EXPANSION_IO42
Routing:
- net Net-(U2-LED+): track 16.1 -> 73.5 mm, vias 2 -> 4
- net /EXPANSION_IO36: track 98.4 -> 66.4 mm
- net /EXPANSION_IO37: track 112.6 -> 81.7 mm
- net /EXPANSION_IO35: track 75.4 -> 48.8 mm
- net Net-(U2-V0): track 35.1 -> 61.4 mm
- net /EXPANSION_IO40: track 30.8 -> 15.1 mm, vias 1 -> 0
- net /EXPANSION_IO38: track 30.4 -> 17.8 mm, vias 1 -> 0
- net /EXPANSION_IO1: track 32.9 -> 20.4 mm
- net /EXPANSION_IO41: track 31.1 -> 41.9 mm
- net /STM32_BOOT0: track 39.3 -> 47.4 mm
- net /EXPANSION_IO2: track 29.8 -> 23.3 mm
- net /STM32_SWDIO: track 53.3 -> 49.4 mm
- net /EXPANSION_IO42: track 33.1 -> 36.2 mm
- net /STM32_SWCLK: track 53.4 -> 50.7 mm
- net /ENCODER_SCL: track 23.6 -> 21.9 mm, vias 0 -> 2
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Other:
- board text added: "STATUS: SPINNING ███████████████ | 15s/30s SETUP: 30s | 4K RPM"
- board text removed: "SPINNING - RPM: 4K RPM | DURATION: 30S"
