File: electronics/io_board/io_board.kicad_sch (KiCad schematic)
At the start: 21 parts, among them SW1 PEC11R-4220F-S0024, SW2 PEC11R-4220F-S0024, SW3 MX1A-11NW, SW4 MX1A-11NW, U1 AFD01-S35FCA-00, U2 HS1602A-B, U3 ZX-PZ1.27-2-5PZZ

Commit message: fix
Parts:
- removed C29: 1u, Capacitor_SMD:C_0402_1005Metric, symbol Device:C
- added C1: 100n, Capacitor_SMD:C_0402_1005Metric, symbol Device:C
Connections:
- net STM32-BOOT0 is gone; now on net STM32_BOOT0: U1.23
- net STM32-SWCLK is gone; now on net STM32_SWCLK: U1.22
- net STM32-SWDIO is gone; now on net STM32_SWDIO: U1.21
- net +3V3: now also C56.1, U3.7, C1.1
- net EXPANSION_IO1: now also U2.4 (RS)
- net EXPANSION_IO10: now also U3.8; no longer SW1.1 (A)
- net EXPANSION_IO11: now also U3.5; no longer SW1.3 (B)
- net EXPANSION_IO12: now also U3.3; no longer SW1.4 (1)
- net EXPANSION_IO13: now also SW1.4 (1); no longer SW2.1 (A)
- net EXPANSION_IO14: now also SW1.1 (A); no longer SW2.3 (B)
- net EXPANSION_IO2: now also U2.6 (E)
- net EXPANSION_IO21: now also SW1.3 (B); no longer SW2.4 (1)
- net EXPANSION_IO35: now also SW2.4 (1); no longer U2.14 (DB7)
- net EXPANSION_IO36: now also SW2.1 (A); no longer U2.13 (DB6)
- net EXPANSION_IO37: now also SW2.3 (B); no longer U2.12 (DB5)
- net EXPANSION_IO38: now also U2.12 (DB5); no longer U2.11 (DB4)
- net EXPANSION_IO40: now also U2.11 (DB4); no longer U2.6 (E)
- net EXPANSION_IO41: now also U2.13 (DB6); no longer U2.4 (RS)
- net EXPANSION_IO42: now also U2.14 (DB7)
- net EXPANSION_IO45: now also R1.2, SW4.1; no longer BUZZER1.1 (+)
- net EXPANSION_IO47: now also BUZZER1.1 (+); no longer R38.2, SW3.1
- net EXPANSION_IO48: now also R38.2, SW3.1; no longer R1.2, SW4.1
- net GND: now also C56.2, U3.10, U3.9, C1.2
- net VBUS: now also U3.6
- net STM32_BOOT0: now reaches U3.1
- net STM32_SWCLK: now reaches U3.2
- net STM32_SWDIO: now reaches U3.4
Other:
- moved on the sheet: C56, U3

Commit message: fix
Connections:
- net +3V3: now also U3.4; no longer U3.7
- net EXPANSION_IO10: now also U3.9; no longer U3.8
- net EXPANSION_IO11: now also U3.7; no longer U3.5
- net EXPANSION_IO12: now also U3.5; no longer U3.3
- net GND: now also U3.1, U3.2; no longer U3.10, U3.9
- net STM32_BOOT0: now also U3.3; no longer U3.1
- net STM32_SWCLK: now also U3.8; no longer U3.2
- net STM32_SWDIO: now also U3.10; no longer U3.4
Other:
- moved on the sheet: U3

Commit message: fix
Connections:
- net EXPANSION_IO1: now also U2.12 (DB5); no longer U2.4 (RS)
- net EXPANSION_IO2: now also U2.11 (DB4); no longer U2.6 (E)
- net EXPANSION_IO38: now also U2.13 (DB6); no longer U2.12 (DB5)
- net EXPANSION_IO40: now also U2.14 (DB7); no longer U2.11 (DB4)
- net EXPANSION_IO41: now also U2.4 (RS); no longer U2.13 (DB6)
- net EXPANSION_IO42: now also U2.6 (E); no longer U2.14 (DB7)
Changed lines of the file:
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@@
-		)
-	)
-	(label "EXPANSION_IO41"
-		(at 157.48 121.92 0)
-		(effects
-			(font
-				(size 1.27 1.27)
-			)
-			(justify left bottom)
 		)
 	)
@@
 	)
 	(label "EXPANSION_IO1"
-		(at 157.48 144.78 0)
+		(at 157.48 124.46 0)
 		(effects
 			(font
@@
 	)
 	(label "EXPANSION_IO40"
-		(at 157.48 127 0)
+		(at 157.48 119.38 0)
 		(effects
 			(font
@@
 	)
 	(label "EXPANSION_IO2"
-		(at 157.48 139.7 0)
+		(at 157.48 127 0)
 		(effects
 			(font
@@
 	)
 	(label "EXPANSION_IO42"
-		(at 157.48 119.38 0)
+		(at 157.48 139.7 0)
 		(effects
 			(font
@@
 		)
 	)
+	(label "EXPANSION_IO38"
+		(at 157.48 121.92 0)
+		(effects
+			(font
+				(size 1.27 1.27)
+			)
+			(justify left bottom)
+		)
+	)
 	(label "EXPANSION_IO42"
 		(at 83.82 127 180)
@@
 		)
 	)
-	(label "EXPANSION_IO38"
-		(at 157.48 124.46 0)
-		(effects
-			(font
+	(label "EXPANSION_IO41"
+		(at 157.48 144.78 0)
+		(effects
+			(font
